Commit message: bigrdigr_gazebo test launch files

File: src/bigrdigr_description/urdf/bigrdigr.gazebo.xacro (robot description, xacro)
@@ -1,9 +1,6 @@
 <?xml version="1.0"?>
-<robot name="digr" xmlns:xacro="https://www.ros.org/wiki/xacro">
+<robot name="bigrdigr" xmlns:xacro="https://www.ros.org/wiki/xacro">
 <xacro:property name="imu_visual" value="false"/>
-<xacro:property name="pseye_FOV" value=""/> <!--56 or 75 degrees, need rad-->
-	<!--<gazebo reference="world_origin">
-		<turnGravityOff>false</turnGravityOff>
-	</gazebo-->
+<xacro:property name="pseye_FOV" value="1.309"/> <!--56 or 75 degrees, need rad-->
 <!-- ToDo
 Pseye camera sensors
@@ -15,6 +12,10 @@
 explore other plugins
 -->
+	<gazebo reference="world_origin">
+		<turnGravityOff>false</turnGravityOff>
+	</gazebo>
 	<gazebo reference="base_link">
 		<material>Gazebo/LightGrey</material>
+		<turnGravityOff>false</turnGravityOff>
 	</gazebo>
 	<gazebo reference="front_left_wheel">
@@ -24,5 +25,5 @@
 		<kd>1.0</kd>
 		<minDepth>0.001</minDepth>
-		<maxVel>1707</maxVel>
+		<maxVel>1</maxVel>
 		<fdir1>1 0 0</fdir1>
 		<material>Gazebo/FlatBlack</material>
@@ -34,5 +35,5 @@
 		<kd>1.0</kd>
 		<minDepth>0.001</minDepth>
-		<maxVel>1707</maxVel>
+		<maxVel>1</maxVel>
 		<fdir1>1 0 0</fdir1>
 		<material>Gazebo/FlatBlack</material>
@@ -44,5 +45,5 @@
 		<kd>1.0</kd>
 		<minDepth>0.001</minDepth>
-		<maxVel>1707</maxVel>
+		<maxVel>1</maxVel>
 		<fdir1>1 0 0</fdir1>
 		<material>Gazebo/FlatBlack</material>
@@ -54,13 +55,13 @@
 		<kd>1.0</kd>
 		<minDepth>0.001</minDepth>
-		<maxVel>1707</maxVel>
-		<fdir1>1 0 0</fdir1>
-		<material>Gazebo/FlatBlack</material>
-	</gazebo>
-<!--	<gazebo>
+		<maxVel>1</maxVel>
+		<fdir1>1 0 0</fdir1>
+		<material>Gazebo/FlatBlack</material>
+	</gazebo>
+	<gazebo>
 		<plugin name="gazebo_ros_control" filename="libgazebo_ros_control.so">
-			<robotNamespce>/</robotNamespace>
+			<robotNamespace>/</robotNamespace>
 		</plugin>
-	</gazebo>-->
+	</gazebo>
 <!-- Cameras-->
 	<gazebo reference="pseye_camera1">
@@ -224,5 +225,5 @@
 	</gazebo>
 	<!-- IMU support -->
-	<gazebo>
+	<!-- <gazebo>
 		<plugin name="imu_plugin" filename="libgazebo_ros_imu.so">
 			<alwaysOn>true</alwaysOn>
@@ -251,4 +252,4 @@
 			</imu>
 		</plugin>
-	</gazebo>
+	</gazebo> -->
 </robot>

File: src/bigrdigr_description/urdf/bigrdigr.urdf.xacro (robot description, xacro)
@@ -1,6 +1,6 @@
 <?xml version="1.0" ?>
-<robot name="digr" xmlsn:xacro="http://ros.org/wiki/xacro">
-	<xacro:include filename="$(find description)/urdf/common_properties.xacro"/>
-	<xacro:include filename="$(find description)/urdf/digr.gazebo.xacro"/>
+<robot name="bigrdigr" xmlns:xacro="https://www.ros.org/wiki/xacro">
+	<!-- <xacro:include filename="$(find description)/urdf/common_properties.xacro"/> -->
+	<xacro:include filename="$(find bigrdigr_description)/urdf/bigrdigr.gazebo.xacro"/>
 	<!-- Define colors -->
 	<!-- All units in meters, kg, seconds, rads -->
@@ -45,5 +45,5 @@
 	<link name="world_origin">
 	<joint name="base_footprint_joint" type="fixed">
-		<origin xyz="0 0 ${wheel_radius - base_hight_to_wheel_origin}" rpy="0 0 0" />
+		<origin xyz="0 0 ${wheel_radius - base_height_origin_to_wheel_origin}" rpy="0 0 0" />
 		<parent link="world_origin" />
 		<child link="base_link" />
@@ -72,5 +72,5 @@
 		<parent link="base_link"/>
 		<child link="front_left_wheel"/>
-		<origin xyz="${base_x_origin_to_wheel} ${base_y_origin_to_wheel_origin} 0" rpy="0 0 0"/>
+		<origin xyz="${base_x_origin_to_wheel_origin} ${base_y_origin_to_wheel_origin} 0" rpy="0 0 0"/>
 		<dynamics damping="0.5" friction="0.1"/> <!-- get real later-->
 		<limit effort="1000" velocity="10"/> <!-- simmulate motors, max velocity and max joint effort -->
@@ -102,5 +102,5 @@
 		<parent link="base_link"/>
 		<child link="front_right_wheel"/>
-		<origin xyz="${base_x_origin_to_wheel} ${-base_y_origin_to_wheel_origin} 0" rpy="0 0 0"/>
+		<origin xyz="${base_x_origin_to_wheel_origin} ${-base_y_origin_to_wheel_origin} 0" rpy="0 0 0"/>
 		<dynamics damping="0.5" friction="0.1"/> <!-- get real later-->
 		<limit effort="1000" velocity="10"/> <!-- simmulate motors, max velocity and max joint effort -->
@@ -131,5 +131,5 @@
 		<parent link="base_link"/>
 		<child link="back_left_wheel"/>
-		<origin xyz="${-base_x_origin_to_wheel} ${base_y_origin_to_wheel_origin} 0" rpy="0 0 0"/>
+		<origin xyz="${-base_x_origin_to_wheel_origin} ${base_y_origin_to_wheel_origin} 0" rpy="0 0 0"/>
 		<dynamics damping="0.5" friction="0.1"/> <!-- get real later-->
 		<limit effort="1000" velocity="10"/> <!-- simmulate motors, max velocity and max joint effort -->
@@ -160,5 +160,5 @@
 		<parent link="base_link"/>
 		<child link="back_right_wheel"/>
-		<origin xyz="${-base_x_origin_to_wheel} ${-base_y_origin_to_wheel_origin} 0" rpy="0 0 0"/>
+		<origin xyz="${-base_x_origin_to_wheel_origin} ${-base_y_origin_to_wheel_origin} 0" rpy="0 0 0"/>
 		<dynamics damping="0.5" friction="0.1"/> <!-- get real later-->
 		<limit effort="1000" velocity="10"/> <!-- simmulate motors, max velocity and max joint effort -->
@@ -187,9 +187,9 @@
 	</link>
 	<!-- IMU -->
-	<joint name="imu_joint" type="fixed">
+	<!-- <joint name="imu_joint" type="fixed">
 		<axis rpy="0 0 0" xyz="0 1 0"/>
 		<parent link="base_link" />
 		<child link="imu_link" />
-		<origin xyz="0 0 ${base_height + ium_height/2.0}" rpy="0 0 0" />
+		<origin xyz="0 0 ${base_height + imu_height/2.0}" rpy="0 0 0" />
 	</joint>
 	<link name="imu_link">
@@ -207,5 +207,5 @@
 			</geometry>
 		</collision>
-	</link>
+	</link> -->
 <!--PSeye Cameras. One in each top corner -->
 <!--Top right camera -->

Commit message: bigrdigr_gazebo launch basic robot + test world

File: src/bigrdigr_description/urdf/bigrdigr.gazebo.xacro (robot description, xacro)
@@ -1,4 +1,7 @@
 <?xml version="1.0"?>
 <robot name="bigrdigr" xmlns:xacro="https://www.ros.org/wiki/xacro">
+<xacro:property name="cam_ambient" value="0.3 0 0 1"/>
+<xacro:property name="cam_diffuse" value="0.5 0 0 1"/>
+<xacro:property name="cam_emissive" value="0.4 0 0 1"/>
 <xacro:property name="imu_visual" value="false"/>
 <xacro:property name="pseye_FOV" value="1.309"/> <!--56 or 75 degrees, need rad-->
@@ -16,5 +19,13 @@
 	</gazebo>
 	<gazebo reference="base_link">
-		<material>Gazebo/LightGrey</material>
+		<!-- <material>Gazebo/Grey</material> -->
+		<visual>
+			<material>
+				<ambient>0.5 0.5 0.5 1</ambient> <!--rgb with no light-->
+				<diffuse>0.8 0.8 0.8 1</diffuse> <!--rgb under white light-->
+				<specular>0 0 0 0</specular> <!--Not working yet in gazebo-->
+				<emissive>0 0 0 1</emissive> <!--rgb emitted-->
+			</material>
+		</visual>
 		<turnGravityOff>false</turnGravityOff>
 	</gazebo>
@@ -66,8 +77,17 @@
 <!-- Cameras-->
 	<gazebo reference="pseye_camera1">
+		<!-- <material>Gazebo/Red</material> -->
+		<visual>
+			<material>
+				<ambient>${cam_ambient}</ambient>
+				<diffuse>${cam_diffuse}</diffuse>
+				<specular>0 0 0 0</specular>
+				<emissive>${cam_emissive}</emissive>
+			</material>
+		</visual>
 		<sensor type="camera" name="cam1">
 			<update_rate>120</update_rate> <!--fps? -->
 			<camera name="front_left">
-				<horizizontal_fov>${pseye_FOV}</horizizontal_fov> <!-- -->
+				<horizontal_fov>${pseye_FOV}</horizontal_fov>
 				<image>
 					<width>320</width>
@@ -104,8 +124,17 @@
 	</gazebo>
 	<gazebo reference="pseye_camera2">
+		<!-- <material>Gazebo/Red</material> -->
+		<visual>
+			<material>
+				<ambient>${cam_ambient}</ambient>
+				<diffuse>${cam_diffuse}</diffuse>
+				<specular>0 0 0 0</specular>
+				<emissive>${cam_emissive}</emissive>
+			</material>
+		</visual>
 		<sensor type="camera" name="cam2">
 			<update_rate>120</update_rate> <!--fps? -->
 			<camera name="front_left">
-				<horizizontal_fov>${pseye_FOV}</horizizontal_fov> <!-- -->
+				<horizontal_fov>${pseye_FOV}</horizontal_fov>
 				<image>
 					<width>320</width>
@@ -142,8 +171,17 @@
 	</gazebo>
 	<gazebo reference="pseye_camera3">
+		<!-- <material>Gazebo/Red</material> -->
+		<visual>
+			<material>
+				<ambient>${cam_ambient}</ambient>
+				<diffuse>${cam_diffuse}</diffuse>
+				<specular>0 0 0 0</specular>
+				<emissive>${cam_emissive}</emissive>
+			</material>
+		</visual>
 		<sensor type="camera" name="cam1">
 			<update_rate>120</update_rate> <!--fps? -->
 			<camera name="front_left">
-				<horizizontal_fov>${pseye_FOV}</horizizontal_fov> <!-- -->
+				<horizontal_fov>${pseye_FOV}</horizontal_fov>
 				<image>
 					<width>320</width>
@@ -180,8 +218,17 @@
 	</gazebo>
 	<gazebo reference="pseye_camera4">
+		<!-- <material>Gazebo/Red</material> -->
+		<visual>
+			<material>
+				<ambient>${cam_ambient}</ambient>
+				<diffuse>${cam_diffuse}</diffuse>
+				<specular>0 0 0 0</specular>
+				<emissive>${cam_emissive}</emissive>
+			</material>
+		</visual>
 		<sensor type="camera" name="cam4">
 			<update_rate>120</update_rate> <!--fps? -->
 			<camera name="front_left">
-				<horizizontal_fov>${pseye_FOV}</horizizontal_fov> <!-- -->
+				<horizontal_fov>${pseye_FOV}</horizontal_fov>
 				<image>
 					<width>320</width>
@@ -222,5 +269,5 @@
 			<visualize>${imu_visual}</visualize>
 		</sensor>
-		<materal>Gazebo/FlatBlack</materal>
+		<material>Gazebo/FlatBlack</material>
 	</gazebo>
 	<!-- IMU support -->

File: src/bigrdigr_description/urdf/bigrdigr.urdf.xacro (robot description, xacro)
@@ -3,5 +3,4 @@
 	<!-- <xacro:include filename="$(find description)/urdf/common_properties.xacro"/> -->
 	<xacro:include filename="$(find bigrdigr_description)/urdf/bigrdigr.gazebo.xacro"/>
-	<!-- Define colors -->
 	<!-- All units in meters, kg, seconds, rads -->
 	<!-- Equation for inertial matrix of box/prisim -->
@@ -43,5 +42,5 @@
 	<!-- world_origin is a fictitious link(frame) that is on the ground right below base_link origin -->
 	<!-- z axis is height -->
-	<link name="world_origin">
+	<link name="world_origin"/>
 	<joint name="base_footprint_joint" type="fixed">
 		<origin xyz="0 0 ${wheel_radius - base_height_origin_to_wheel_origin}" rpy="0 0 0" />
@@ -53,7 +52,7 @@
 			<origin xyz="0 0 ${base_height/2.0}" rpy="0 0 0"/>
 			<geometry>
-				<mesh filename="~/NASA_ws/digr/description/meshes/base_link.stl" scale="0.001 0.001 0.001"/>
-			</geometry>
-			<material name="grey"/>
+				<box size=" ${base_length} ${base_width} ${base_height}" />
+				<!-- <mesh filename="~/NASA_ws/digr/description/meshes/base_link.stl" scale="0.001 0.001 0.001"/> -->
+			</geometry>
 		</visual>
 		<collision>
@@ -95,5 +94,5 @@
 			<origin xyz="0 0 0" />
 			<mass value="${wheel_mass}" />
-			<cylinder_inertial_matrix m="${wheel_mass}" h="${wheel_height}" r="${wheel_radius}"/>
+			<cylinder_inertia m="${wheel_mass}" h="${wheel_height}" r="${wheel_radius}"/>
 		</inertial>
 	</link>
@@ -125,5 +124,5 @@
 			<origin xyz="0 0 0" />
 			<mass value="${wheel_mass}" />
-			<cylinder_inertial_matrix m="${wheel_mass}" h="${wheel_height}" r="${wheel_radius}"/>
+			<cylinder_inertia m="${wheel_mass}" h="${wheel_height}" r="${wheel_radius}"/>
 		</inertial>
 	</link>
@@ -154,5 +153,5 @@
 			<origin xyz="0 0 0" />
 			<mass value="${wheel_mass}" />
-			<cylinder_inertial_matrix m="${wheel_mass}" h="${wheel_height}" r="${wheel_radius}"/>
+			<cylinder_inertia m="${wheel_mass}" h="${wheel_height}" r="${wheel_radius}"/>
 		</inertial>
 	</link>
@@ -183,5 +182,5 @@
 			<origin xyz="0 0 0" />
 			<mass value="${wheel_mass}" />
-			<cylinder_inertial_matrix m="${wheel_mass}" h="${wheel_height}" r="${wheel_radius}"/>
+			<cylinder_inertia m="${wheel_mass}" h="${wheel_height}" r="${wheel_radius}"/>
 		</inertial>
 	</link>
@@ -222,5 +221,4 @@
 					<box size="${pseye_camera_length} ${pseye_camera_width} ${pseye_camera_height}"/>
 				</geometry>
-				<materal name="blue"/>
 			</visual>
 			<collision>
@@ -232,5 +230,5 @@
 		</link>
 <!--Top left camera -->
-	<joint name="camera1_joint" type="fixed">
+	<joint name="camera2_joint" type="fixed">
 		<axis xyz="0 1 0" />
 		<origin xyz="${-base_width/2} ${base_length/2.0} ${base_height}" rpy="0 0 0"/>
@@ -244,5 +242,4 @@
 			<box size="${pseye_camera_length} ${pseye_camera_width} ${pseye_camera_height}"/>
 		</geometry>
-		<materal name="blue"/>
 	</visual>
 	<collision>
@@ -254,5 +251,5 @@
 </link>
 <!--Back right camera -->
-	<joint name="camera1_joint" type="fixed">
+	<joint name="camera3_joint" type="fixed">
 		<axis xyz="0 1 0" />
 		<origin xyz="${base_width/2} ${-base_length/2.0} ${base_height}" rpy="0 0 0"/>
@@ -266,5 +263,4 @@
 				<box size="${pseye_camera_length} ${pseye_camera_width} ${pseye_camera_height}"/>
 			</geometry>
-			<materal name="blue"/>
 		</visual>
 		<collision>
@@ -276,5 +272,5 @@
 	</link>
 <!--Back left camera -->
-		<joint name="camera1_joint" type="fixed">
+		<joint name="camera4_joint" type="fixed">
 			<axis xyz="0 1 0" />
 			<origin xyz="${-base_width/2} ${-base_length/2.0} ${base_height}" rpy="0 0 0"/>
@@ -288,5 +284,4 @@
 					<box size="${pseye_camera_length} ${pseye_camera_width} ${pseye_camera_height}"/>
 				</geometry>
-				<materal name="blue"/>
 			</visual>
 			<collision>
@@ -297,5 +292,4 @@
 			</collision>
 		</link>
-	</link>
 </robot>
 <!-- 4 cams, IMU -->

Commit message: bigrdigr_control testing ros_control files

File: src/bigrdigr_description/urdf/bigrdigr.gazebo.xacro (robot description, xacro)
@@ -72,5 +72,5 @@
 	<gazebo>
 		<plugin name="gazebo_ros_control" filename="libgazebo_ros_control.so">
-			<robotNamespace>/</robotNamespace>
+			<robotNamespace>/bigrdigr</robotNamespace>
 		</plugin>
 	</gazebo>

File: src/bigrdigr_description/urdf/bigrdigr.urdf.xacro (robot description, xacro)
@@ -97,4 +97,14 @@
 		</inertial>
 	</link>
+	<transmission name="front_left_wheel_trans">
+		<type>transmission_interface/SimpleTransmission</type>
+		<joint name="front_left_wheel_joint">
+			<hardwareInterface>EffortJointInterface</hardwareInterface>
+		</joint>
+		<actuator name="front_left_wheel_motor">
+			<hardwareInterface>EffortJointInterface</hardwareInterface>
+			<mechanicalReduction>1</mechanicalReduction>
+		</actuator>
+	</transmission>
 	<!-- Transmission sims motor control -->
 	<joint name="front_right_wheel_joint" type="continuous">
@@ -127,4 +137,14 @@
 		</inertial>
 	</link>
+	<transmission name="front_left_wheel_trans">
+		<type>transmission_interface/SimpleTransmission</type>
+		<joint name="front_left_wheel_joint">
+			<hardwareInterface>EffortJointInterface</hardwareInterface>
+		</joint>
+		<actuator name="front_left_wheel_motor">
+			<hardwareInterface>EffortJointInterface</hardwareInterface>
+			<mechanicalReduction>1</mechanicalReduction>
+		</actuator>
+	</transmission>
 	<joint name="back_left_wheel_joint" type="continuous">
 		<parent link="base_link"/>
@@ -156,4 +176,14 @@
 		</inertial>
 	</link>
+	<transmission name="front_left_wheel_trans">
+		<type>transmission_interface/SimpleTransmission</type>
+		<joint name="front_left_wheel_joint">
+			<hardwareInterface>EffortJointInterface</hardwareInterface>
+		</joint>
+		<actuator name="front_left_wheel_motor">
+			<hardwareInterface>EffortJointInterface</hardwareInterface>
+			<mechanicalReduction>1</mechanicalReduction>
+		</actuator>
+	</transmission>
 	<joint name="back_right_wheel_joint" type="continuous">
 		<parent link="base_link"/>
@@ -185,4 +215,14 @@
 		</inertial>
 	</link>
+	<transmission name="front_left_wheel_trans">
+		<type>transmission_interface/SimpleTransmission</type>
+		<joint name="front_left_wheel_joint">
+			<hardwareInterface>EffortJointInterface</hardwareInterface>
+		</joint>
+		<actuator name="front_left_wheel_motor">
+			<hardwareInterface>EffortJointInterface</hardwareInterface>
+			<mechanicalReduction>1</mechanicalReduction>
+		</actuator>
+	</transmission>
 	<!-- IMU -->
 	<!-- <joint name="imu_joint" type="fixed">
