Commit message: bigrdigr_input simple velocity publishing

File: src/bigrdigr_description/urdf/bigrdigr.gazebo.xacro (robot description, xacro)
@@ -1,8 +1,5 @@
 <?xml version="1.0"?>
 <robot name="bigrdigr" xmlns:xacro="https://www.ros.org/wiki/xacro">
-<xacro:property name="cam_ambient" value="0.3 0 0 1"/>
-<xacro:property name="cam_diffuse" value="0.5 0 0 1"/>
-<xacro:property name="cam_emissive" value="0.4 0 0 1"/>
-<xacro:property name="imu_visual" value="false"/>
+<xacro:property name="imu_visual" value="true"/>
 <xacro:property name="pseye_FOV" value="1.309"/> <!--56 or 75 degrees, need rad-->
 <!-- ToDo
@@ -19,13 +16,5 @@
 	</gazebo>
 	<gazebo reference="base_link">
-		<!-- <material>Gazebo/Grey</material> -->
-		<visual>
-			<material>
-				<ambient>0.5 0.5 0.5 1</ambient> <!--rgb with no light-->
-				<diffuse>0.8 0.8 0.8 1</diffuse> <!--rgb under white light-->
-				<specular>0 0 0 0</specular> <!--Not working yet in gazebo-->
-				<emissive>0 0 0 1</emissive> <!--rgb emitted-->
-			</material>
-		</visual>
+		<material>Gazebo/Grey</material>
 		<turnGravityOff>false</turnGravityOff>
 	</gazebo>
@@ -77,13 +66,5 @@
 <!-- Cameras-->
 	<gazebo reference="pseye_camera1">
-		<!-- <material>Gazebo/Red</material> -->
-		<visual>
-			<material>
-				<ambient>${cam_ambient}</ambient>
-				<diffuse>${cam_diffuse}</diffuse>
-				<specular>0 0 0 0</specular>
-				<emissive>${cam_emissive}</emissive>
-			</material>
-		</visual>
+		<material>Gazebo/Red</material>
 		<sensor type="camera" name="cam1">
 			<update_rate>120</update_rate> <!--fps? -->
@@ -124,13 +105,5 @@
 	</gazebo>
 	<gazebo reference="pseye_camera2">
-		<!-- <material>Gazebo/Red</material> -->
-		<visual>
-			<material>
-				<ambient>${cam_ambient}</ambient>
-				<diffuse>${cam_diffuse}</diffuse>
-				<specular>0 0 0 0</specular>
-				<emissive>${cam_emissive}</emissive>
-			</material>
-		</visual>
+		<material>Gazebo/Red</material>
 		<sensor type="camera" name="cam2">
 			<update_rate>120</update_rate> <!--fps? -->
@@ -171,13 +144,5 @@
 	</gazebo>
 	<gazebo reference="pseye_camera3">
-		<!-- <material>Gazebo/Red</material> -->
-		<visual>
-			<material>
-				<ambient>${cam_ambient}</ambient>
-				<diffuse>${cam_diffuse}</diffuse>
-				<specular>0 0 0 0</specular>
-				<emissive>${cam_emissive}</emissive>
-			</material>
-		</visual>
+		<material>Gazebo/Red</material>
 		<sensor type="camera" name="cam1">
 			<update_rate>120</update_rate> <!--fps? -->
@@ -218,13 +183,5 @@
 	</gazebo>
 	<gazebo reference="pseye_camera4">
-		<!-- <material>Gazebo/Red</material> -->
-		<visual>
-			<material>
-				<ambient>${cam_ambient}</ambient>
-				<diffuse>${cam_diffuse}</diffuse>
-				<specular>0 0 0 0</specular>
-				<emissive>${cam_emissive}</emissive>
-			</material>
-		</visual>
+		<material>Gazebo/Red</material>
 		<sensor type="camera" name="cam4">
 			<update_rate>120</update_rate> <!--fps? -->
@@ -265,38 +222,22 @@
 	</gazebo>
 	<gazebo reference="imu_link">
+		<gravity>true</gravity>
 		<sensor type="imu" name="imu">
 			<always_on>true</always_on>
+			<update_rate>100</update_rate>
 			<visualize>${imu_visual}</visualize>
-		</sensor>
-		<material>Gazebo/FlatBlack</material>
-	</gazebo>
-	<!-- IMU support -->
-	<!-- <gazebo>
-		<plugin name="imu_plugin" filename="libgazebo_ros_imu.so">
-			<alwaysOn>true</alwaysOn>
-			<bodyName>imu_link</bodyName>
-			<frameName>imu_link</frameName>
-			<topicName>imu</topicName>
-			<serviceName>imu_service</serviceName>
-			<gaussianNoise>0.0</gaussianNoise>
-			<updateRate>200</updateRate>
-			<imu>
-				<noise>
-					<type>gaussian</type>
-					<rate>
-						<mean>0.0</mean>
-						<stddev>2e-4</stddev>
-						<bias_mean>0.0000075</bias_mean>
-						<bias_stddev>0.0000008</bias_stddev>
-					</rate>
-					<accel>
-						<mean>0.0</mean>
-						<stddev>1.7e-2</stddev>
-						<bias_mean>0.1</bias_mean>
-						<bias_stddev>0.001</bias_stddev>
-					</accel>
-				</noise>
-			</imu>
-		</plugin>
-	</gazebo> -->
+			<topic>imu_data</topic>
+			<plugin filename="libgazebo_ros_imu_sensor.so" name="imu_plugin">
+				<topicName>imu</topicName>
+				<bodyName>imu_link</bodyName>
+				<updateRateHZ>10.0</updateRateHZ>
+				<gaussianNoise>0.0</gaussianNoise>
+				<xyzOffset>0 0 0</xyzOffset>
+				<rpyOffset>0 0 0</rpyOffset>
+				<frameName>imu_link</frameName>
+			</plugin>
+			<pose>0 0 0 0 0 0</pose>
+		</sensor>
+		<material>Gazebo/FlatBlack</material>
+	</gazebo>
 </robot>

File: src/bigrdigr_description/urdf/bigrdigr.urdf.xacro (robot description, xacro)
@@ -68,4 +68,18 @@
 		</inertial>
 	</link>
+	<joint name="scoop_joint" type="fixed">
+		<parent link="base_link"/>
+		<child link="scoop_link"/>
+		<origin xyz="${base_length/2} 0 ${base_height/2}" rpy="0 0 0"/>
+	</joint>
+	<link name="scoop_link">
+		<visual>
+			<origin xyz="0 0 0" rpy="0 0 0"/>
+			<geometry>
+				<box size="0.01 0.2 0.2"/>
+			</geometry>
+			<material name="purple"/>
+		</visual>
+	</link>
 	<joint name="front_left_wheel_joint" type="continuous">
 		<parent link="base_link"/>

File: src/bigrdigr_description/urdf/bigrdigr1.gazebo.xacro (robot description, xacro)
@@ -1,5 +1,5 @@
 <?xml version="1.0"?>
 <robot name="bigrdigr" xmlns:xacro="https://www.ros.org/wiki/xacro">
-<xacro:property name="imu_visual" value="false"/>
+<xacro:property name="imu_visual" value="true"/>
 <xacro:property name="pseye_FOV" value="1.309"/> <!--56 or 75 degrees, need rad-->
 <!-- ToDo
@@ -8,13 +8,12 @@
 real sense sensors
 decawave sensors (1001) (talks between robot and base station for speed)
-gps (decawave)
 wheel odometry (encoders, handleed in ros)
 explore other plugins
 -->
-	<gazebo>
+	<!-- <gazebo>
 		<plugin name="gazebo_ros_control" filename="libgazebo_ros_control.so">
 			<robotNamespace>/bigrdigr</robotNamespace>
 		</plugin>
-	</gazebo>
+	</gazebo> -->
 	<gazebo reference="world_origin">
 		<turnGravityOff>false</turnGravityOff>
@@ -24,4 +23,8 @@
 		<turnGravityOff>false</turnGravityOff>
 	</gazebo>
+	<gazebo reference="scoop_link">
+		<material>Gazebo/Purple</material>
+		<turnGravityOff>false</turnGravityOff>
+	</gazebo>
 	<gazebo reference="front_left_wheel">
 		<mu1>0.3</mu1>
@@ -221,9 +224,72 @@
 	</gazebo>
 	<gazebo reference="imu_link">
+		<gravity>true</gravity>
 		<sensor type="imu" name="imu">
 			<always_on>true</always_on>
+			<update_rate>100</update_rate>
 			<visualize>${imu_visual}</visualize>
+			<topic>imu_data</topic>
+			<plugin filename="libgazebo_ros_imu_sensor.so" name="imu_plugin">
+				<topicName>imu</topicName>
+				<bodyName>imu_link</bodyName>
+				<updateRateHZ>10.0</updateRateHZ>
+				<gaussianNoise>0.0</gaussianNoise>
+				<xyzOffset>0 0 0</xyzOffset>
+				<rpyOffset>0 0 0</rpyOffset>
+				<frameName>imu_link</frameName>
+			</plugin>
+			<pose>0 0 0 0 0 0</pose>
 		</sensor>
 		<material>Gazebo/Blue</material>
 	</gazebo>
+	<!-- <gazebo>
+	  <plugin name="differential_drive_controller1" filename="libgazebo_ros_diff_drive.so">
+	    <alwaysOn>true</alwaysOn>
+	    <updateRate>100</updateRate>
+	    <leftJoint>front_left_wheel_joint</leftJoint>
+	    <rightJoint>front_right_wheel_joint</rightJoint>
+	    <wheelSeparation>0.5825</wheelSeparation>
+	    <wheelDiameter>0.348</wheelDiameter>
+	    <torque>20</torque>
+	    <commandTopic>cmd_vel</commandTopic>
+	    <odometryTopic>odom</odometryTopic>
+	    <odometryFrame>odom</odometryFrame>
+	    <robotBaseFrame>world_origin</robotBaseFrame>
+			<legacyMode>false</legacyMode>
+	  </plugin>
+	</gazebo>
+	<gazebo>
+	  <plugin name="differential_drive_controller2" filename="libgazebo_ros_diff_drive.so">
+	    <alwaysOn>true</alwaysOn>
+	    <updateRate>100</updateRate>
+	    <leftJoint>back_left_wheel_joint</leftJoint>
+	    <rightJoint>back_right_wheel_joint</rightJoint>
+	    <wheelSeparation>0.5825</wheelSeparation>
+	    <wheelDiameter>0.348</wheelDiameter>
+	    <torque>20</torque>
+	    <commandTopic>cmd_vel</commandTopic>
+	    <odometryTopic>odom</odometryTopic>
+	    <odometryFrame>odom</odometryFrame>
+	    <robotBaseFrame>world_origin</robotBaseFrame>
+			<legacyMode>false</legacyMode>
+	  </plugin>
+	</gazebo> -->
+	<gazebo>
+	  <plugin name="skid_steer_drive_controller" filename="libgazebo_ros_skid_steer_drive.so">
+	    <updateRate>100.0</updateRate>
+	    <robotNamespace>/bigrdigr</robotNamespace>
+			<commandTopic>/cmd_vel</commandTopic>
+			<odometryTopic>/odom</odometryTopic>
+	    <leftFrontJoint>front_left_wheel_joint</leftFrontJoint>
+	    <rightFrontJoint>front_right_wheel_joint</rightFrontJoint>
+	    <leftRearJoint>back_left_wheel_joint</leftRearJoint>
+	    <rightRearJoint>back_right_wheel_joint</rightRearJoint>
+	    <wheelSeparation>0.5825</wheelSeparation>
+	    <wheelDiameter>0.348</wheelDiameter>
+	    <robotBaseFrame>base_link</robotBaseFrame>
+	    <torque>20</torque>
+	    <broadcastTF>true</broadcastTF>
+			<legacyMode>false</legacyMode>
+	  </plugin>
+	</gazebo>
 </robot>
