Commit message: my code sucks, but it shouldn't be hard to fix and I have an exam tomorrow so I will fix it later

File: src/bigrdigr_description/urdf/wheel.urdf.xacro (robot description, xacro)
@@ -41,5 +41,15 @@
     </joint>
 	</xacro:macro>
-  <xacro:macro name="null">
+  <xacro:macro name="wheel_trans" params="prefix">
+    <transmission name="${prefix}_wheel_trans">
+      <type>transmission_interface/SimpleTransmission</type>
+      <joint name="${prefix}_wheel_joint">
+        <hardwareInterface>EffortJointInterface</hardwareInterface>
+      </joint>
+      <actuator name="${prefix}_wheel_motor">
+        <hardwareInterface>EffortJointInterface</hardwareInterface>
+        <mechanicalReduction>1</mechanicalReduction>
+      </actuator>
+    </transmission>
   </xacro:macro>
 </robot>
