Commit message: bigrdigr_description initial commit of files

File: src/bigrdigr_description/urdf/bigrdigr.urdf.xacro (robot description, xacro)
@@ -29,4 +29,7 @@
 	<xacro:property name="wheel_height" value="0.15" />
 	<xacro:property name="wheel_mass" value="2" />
+	<xacro:property name="imu_length" value="" />
+	<xacro:property name="imu_width" value="" />
+	<xacro:property name="imu_height" value="" />
 	<!-- World Origin -->
 	<!-- world_origin is a fictitious link(frame) that is on the ground right below base_link origin -->
@@ -176,8 +179,4 @@
 	</link>
 	<!-- IMU -->
-	<!-- Main dimensions: meters, kg, seconds, rads -->
-	<xacro:property name="imu_length" value="" />
-	<xacro:property name="imu_width" value="" />
-	<xacro:property name="imu_height" value="" />
 	<joint name="imu_joint" type="fixed">
 		<axis rpy="0 0 0" xyz="0 1 0"/>

Commit message: bigrdigr_description intial urdf values

File: src/bigrdigr_description/urdf/bigrdigr.urdf.xacro (robot description, xacro)
@@ -50,5 +50,5 @@
 		</visual>
 		<collision>
-			<origin xzy="0 0 ${base_height/2.0}" rpy="0 0 0"/>
+			<origin xyz="0 0 ${base_height/2.0}" rpy="0 0 0"/>
 			<geometry>
 				<box size="${base_length} ${base_width} ${base_width}"/>

File: src/bigrdigr_description/urdf/robot.gazebo.xacro (robot description, xacro)
@@ -1,17 +1,62 @@
 <?xml version="1.0"?>
 <robot name="digr" xmlns:xacro="https://www.ros.org/wiki/xacro">
-	<gazebo reference="world_origin">
+<xacro:property name="imu_visual" value="false"/>
+	<!--<gazebo reference="world_origin">
 		<turnGravityOff>false</turnGravityOff>
-	</gazebo>
+	</gazebo-->
 	<gazebo reference="base_link">
 		<material>Gazebo/LightGrey</material>
-		<turnGravityOff>false</turnGravityOff>
 	</gazebo>
 	<gazebo reference="front_left_wheel">
-		<
-	<gazebo>
+		<mu1>1.0</mu1>
+		<mu2>1.0</mu2>
+		<kp>1000000.0</kp>
+		<kd>1.0</kd>
+		<minDepth>0.001</minDepth>
+		<maxVel>1707</maxVel>
+		<fdir1>1 0 0</fdir1>
+		<material>Gazebo/FlatBlack</material>
+	</gazebo>
+	<gazebo reference="front_right_wheel">
+		<mu1>1.0</mu1>
+		<mu2>1.0</mu2>
+		<kp>1000000.0</kp>
+		<kd>1.0</kd>
+		<minDepth>0.001</minDepth>
+		<maxVel>1707</maxVel>
+		<fdir1>1 0 0</fdir1>
+		<material>Gazebo/FlatBlack</material>
+	</gazebo>
+	<gazebo reference="back_left_wheel">
+		<mu1>1.0</mu1>
+		<mu2>1.0</mu2>
+		<kp>1000000.0</kp>
+		<kd>1.0</kd>
+		<minDepth>0.001</minDepth>
+		<maxVel>1707</maxVel>
+		<fdir1>1 0 0</fdir1>
+		<material>Gazebo/FlatBlack</material>
+	</gazebo>
+	<gazebo reference="back_right_wheel">
+		<mu1>1.0</mu1>
+		<mu2>1.0</mu2>
+		<kp>1000000.0</kp>
+		<kd>1.0</kd>
+		<minDepth>0.001</minDepth>
+		<maxVel>1707</maxVel>
+		<fdir1>1 0 0</fdir1>
+		<material>Gazebo/FlatBlack</material>
+	</gazebo>
+<!--	<gazebo>
 		<plugin name="gazebo_ros_control" filename="libgazebo_ros_control.so">
 			<robotNamespce>/</robotNamespace>
 		</plugin>
+	</gazebo>-->
+	<gazebo reference="imu_link">
+		<sensor type="imu" name="imu">
+			<always_on>true</always_on>
+			<visualize>${imu_visual}</visualize>
+		</sensor>
+		<materal>Gazebo/FlatBlack</materal>
 	</gazebo>
 	<!-- IMU support -->
@@ -23,6 +68,6 @@
 			<topicName>imu</topicName>
 			<serviceName>imu_service</serviceName>
-			<gaussianNoise>    </gaussianNoise>
-			<updateRate>     </updateRate>
+			<gaussianNoise>0.0</gaussianNoise>
+			<updateRate>200</updateRate>
 			<imu>
 				<noise>

Commit message: bigrdigr_description fix urdf typo

File: src/bigrdigr_description/urdf/bigrdigr.urdf.xacro (robot description, xacro)
@@ -7,12 +7,12 @@
 	<!-- Equation for inertial matrix of box/prisim -->
 	<xacro:macro name="box_inertial_matrix" params="m l w h">
-		<inertia ixx="${(m*(w*w+h*h))/12.0}" ixy = "0" ixz = "0"
-				 iyy="${(m*(l*l+h*h))/12.0}" iyz = "0"
+		<inertia ixx="${(m*(w*w+h*h))/12.0}" ixy = "0.0" ixz = "0.0"
+				 iyy="${(m*(l*l+h*h))/12.0}" iyz = "0.0"
 				 izz="${(m*(l*l+w*w))/12.0}" />
 	</xacro:macro>
 	<!-- Equation for inertial matrix of cylinder (rotating around y axis) -->
 	<xacro:macro name="cylinder_inertia" params="m r h">
-		<inertia ixx="${(m*(3*r*r+h*h))/12.0}" ixy = "0" ixz = "0"
-				 iyy="${m*r*r/2}"			   iyz = "0"
+		<inertia ixx="${(m*(3*r*r+h*h))/12.0}" ixy = "0.0" ixz = "0.0"
+				 iyy="${m*r*r/2.0}"			   iyz = "0.0"
 				 izz="${(m*(3*r*r+h*h))/12.0}"  />
 	</xacro:macro>
@@ -22,5 +22,5 @@
 	<xacro:property name="base_length" value="0.740" />
 	<xacro:property name="base_width" value="0.865" />
-	<xacro:property name="base_mass" value="72" />
+	<xacro:property name="base_mass" value="72.0" />
 	<xacro:property name="base_x_origin_to_wheel_origin" value="0.29125" />
 	<xacro:property name="base_y_origin_to_wheel_origin" value="0.190" />
@@ -28,12 +28,20 @@
 	<xacro:property name="wheel_radius" value="0.174" />
 	<xacro:property name="wheel_height" value="0.15" />
-	<xacro:property name="wheel_mass" value="2" />
-	<xacro:property name="imu_length" value="" />
-	<xacro:property name="imu_width" value="" />
-	<xacro:property name="imu_height" value="" />
+	<xacro:property name="wheel_mass" value="2.0" />
+	<xacro:property name="imu_length" value="0.025" />
+	<xacro:property name="imu_width" value="0.025" />
+	<xacro:property name="imu_height" value="0.01" />
+	<xacro:property name="pseye_camera_height" value="0.08" />
+	<xacro:property name="pseye_camera_length" value="0.07" />
+	<xacro:property name="pseye_camera_width" value="0.09" />
+	<!-- 4 top corners-->
+	<!--<xacro:property name="realSense_camera_height" value="0.09" />
+	<xacro:property name="realSense_camera_length" value="0.025" />
+	<xacro:property name="realSense_camera_width" value="0.025" />-->
+ <!--front middle-in, back middle-in, top middle -->
 	<!-- World Origin -->
 	<!-- world_origin is a fictitious link(frame) that is on the ground right below base_link origin -->
 	<!-- z axis is height -->
-	<link name="world_origin"/>
+	<link name="world_origin">
 	<joint name="base_footprint_joint" type="fixed">
 		<origin xyz="0 0 ${wheel_radius - base_hight_to_wheel_origin}" rpy="0 0 0" />
@@ -183,17 +191,110 @@
 		<parent link="base_link" />
 		<child link="imu_link" />
-		<origin rp="0 0 0" xyz="0 0 ${base_height + ium_height/2.0}" />
+		<origin xyz="0 0 ${base_height + ium_height/2.0}" rpy="0 0 0" />
 	</joint>
 	<link name="imu_link">
 		<visual>
+			<origin xyz="0 0 0" rpy="0 0 0" />
 			<geometry>
 				<box size="${imu_length} ${imu_width} ${imu_height}" />
 			</geometry>
-		</visual>
-		<collision>
+			<materal name="purple"/>
+		</visual>
+		<collision>
+			<origin xyz="0 0 0" rpy="0 0 0" />
 			<geometry>
 				<box size="${imu_length} ${imu_width} ${imu_height}" />
 			</geometry>
 		</collision>
+	</link>
+<!--PSeye Cameras. One in each top corner -->
+<!--Top right camera -->
+		<joint name="camera1_joint" type="fixed">
+			<axis xyz="0 1 0" />
+			<origin xyz="${base_width/2} ${base_length/2.0} ${base_height}" rpy="0 0 0"/>
+			<parent link="base_link"/>
+			<child link="pseye_camera1"/>
+		</joint>
+		<link name="pseye_camera1">
+			<visual>
+				<origin xyz="0 0 0" rpy="0 0 0"/>
+				<geometry>
+					<box size="${pseye_camera_length} ${pseye_camera_width} ${pseye_camera_height}"/>
+				</geometry>
+				<materal name="blue"/>
+			</visual>
+			<collision>
+				<origin xyz="0 0 0" rpy="0 0 0" />
+				<geometry>
+					<box size="${pseye_camera_length} ${pseye_camera_width} ${pseye_camera_height}"/>
+				</geometry>
+			</collision>
+		</link>
+<!--Top left camera -->
+	<joint name="camera1_joint" type="fixed">
+		<axis xyz="0 1 0" />
+		<origin xyz="${-base_width/2} ${base_length/2.0} ${base_height}" rpy="0 0 0"/>
+		<parent link="base_link"/>
+		<child link="pseye_camera2"/>
+	</joint>
+<link name="pseye_camera2">
+	<visual>
+		<origin xyz="0 0 0" rpy="0 0 0"/>
+		<geometry>
+			<box size="${pseye_camera_length} ${pseye_camera_width} ${pseye_camera_height}"/>
+		</geometry>
+		<materal name="blue"/>
+	</visual>
+	<collision>
+		<origin xyz="0 0 0" rpy="0 0 0" />
+		<geometry>
+			<box size="${pseye_camera_length} ${pseye_camera_width} ${pseye_camera_height}"/>
+		</geometry>
+	</collision>
+</link>
+<!--Back right camera -->
+	<joint name="camera1_joint" type="fixed">
+		<axis xyz="0 1 0" />
+		<origin xyz="${base_width/2} ${-base_length/2.0} ${base_height}" rpy="0 0 0"/>
+		<parent link="base_link"/>
+		<child link="pseye_camera3"/>
+	</joint>
+	<link name="pseye_camera3">
+		<visual>
+			<origin xyz="0 0 0" rpy="0 0 0"/>
+			<geometry>
+				<box size="${pseye_camera_length} ${pseye_camera_width} ${pseye_camera_height}"/>
+			</geometry>
+			<materal name="blue"/>
+		</visual>
+		<collision>
+			<origin xyz="0 0 0" rpy="0 0 0" />
+			<geometry>
+				<box size="${pseye_camera_length} ${pseye_camera_width} ${pseye_camera_height}"/>
+			</geometry>
+		</collision>
+	</link>
+<!--Back left camera -->
+		<joint name="camera1_joint" type="fixed">
+			<axis xyz="0 1 0" />
+			<origin xyz="${-base_width/2} ${-base_length/2.0} ${base_height}" rpy="0 0 0"/>
+			<parent link="base_link"/>
+			<child link="pseye_camera4"/>
+		</joint>
+		<link name="pseye_camera4">
+			<visual>
+				<origin xyz="0 0 0" rpy="0 0 0"/>
+				<geometry>
+					<box size="${pseye_camera_length} ${pseye_camera_width} ${pseye_camera_height}"/>
+				</geometry>
+				<materal name="blue"/>
+			</visual>
+			<collision>
+				<origin xyz="0 0 0" rpy="0 0 0" />
+				<geometry>
+					<box size="${pseye_camera_length} ${pseye_camera_width} ${pseye_camera_height}"/>
+				</geometry>
+			</collision>
+		</link>
 	</link>
 </robot>

File: src/bigrdigr_description/urdf/robot.gazebo.xacro (robot description, xacro)
@@ -53,4 +53,41 @@
 		</plugin>
 	</gazebo>-->
+<!-- Cameras-->
+	<gazebo reference="pseye_camera1">
+		<sensor type="camera" name="cam1">
+			<update_rate></update_rate>
+			<camera name="front_left">
+				<horizizontal_fov></horizizontal_fov>
+				<image>
+					<width></width>
+					<height></height>
+					<format></format>
+				</image>
+				<clip>
+					<near></near>
+					<far></far>
+				</clip>
+				<noise>
+					<type>gaussian</type>
+					<mean></mean>
+					<stddev></stddev>
+				</noise>
+			</camera>
+			<plugin name="camera_controller" filename="libgazebo_ros_camera.so">
+				<alwaysOn>true</alwaysOn>
+				<updateRate></updateRate>
+				<cameraName></cameraName>
+				<imageTopicName></imageTopicName>
+				<cameraInfoTopicName></cameraInfoTopicName>
+				<frameName>pseye_camera1</frameName>
+				<hackBaseline></hackBaseline>
+				<distortionK1></distortionK1>
+				<distortionK2></distortionK2>
+				<distortionK3></distortionK3>
+				<distortionT1></distortionT1>
+				<distortionT2></distortionT2>
+			</plugin>
+		</sensor>
+	</gazebo>
 	<gazebo reference="imu_link">
 		<sensor type="imu" name="imu">

Commit message: Controllers should work, computer double checking

File: src/bigrdigr_description/urdf/bigrdigr.urdf.xacro (robot description, xacro)
@@ -1,6 +1,5 @@
 <?xml version="1.0" ?>
 <robot name="bigrdigr" xmlns:xacro="https://www.ros.org/wiki/xacro">
-	<!-- <xacro:include filename="$(find description)/urdf/common_properties.xacro"/> -->
-	<xacro:include filename="$(find bigrdigr_description)/urdf/bigrdigr.gazebo.xacro"/>
+	<xacro:include filename="$(find bigrdigr_description)/urdf/bigrdigr1.gazebo.xacro"/>
 	<!-- All units in meters, kg, seconds, rads -->
 	<!-- Equation for inertial matrix of box/prisim -->
@@ -55,4 +54,5 @@
 				<!-- <mesh filename="~/NASA_ws/digr/description/meshes/base_link.stl" scale="0.001 0.001 0.001"/> -->
 			</geometry>
+			<material name="grey"/>
 		</visual>
 		<collision>
@@ -82,5 +82,5 @@
 				<cylinder length="${wheel_height}" radius="${wheel_radius}" />
 			</geometry>
-			<mesh filename="~/NASA_ws/digr/description/meshes/wheel_1.stl" scale="0.001 0.001 0.001"/>
+			<!-- <mesh filename="~/NASA_ws/digr/description/meshes/wheel_1.stl" scale="0.001 0.001 0.001"/> -->
 			<material name="light_black"/>
 		</visual>
@@ -122,5 +122,5 @@
 				<cylinder length="${wheel_height}" radius="${wheel_radius}" />
 			</geometry>
-			<mesh filename="~/NASA_ws/digr/description/meshes/wheel_1.stl" scale="0.001 0.001 0.001"/>
+			<!-- <mesh filename="~/NASA_ws/digr/description/meshes/wheel_1.stl" scale="0.001 0.001 0.001"/> -->
 			<material name="light_black"/>
 		</visual>
@@ -161,5 +161,5 @@
 				<cylinder length="${wheel_height}" radius="${wheel_radius}" />
 			</geometry>
-			<mesh filename="~/NASA_ws/digr/description/meshes/wheel_1.stl" scale="0.001 0.001 0.001"/>
+			<!-- <mesh filename="~/NASA_ws/digr/description/meshes/wheel_1.stl" scale="0.001 0.001 0.001"/> -->
 			<material name="light_black"/>
 		</visual>
@@ -200,5 +200,5 @@
 				<cylinder length="${wheel_height}" radius="${wheel_radius}" />
 			</geometry>
-			<mesh filename="~/NASA_ws/digr/description/meshes/wheel_1.stl" scale="0.001 0.001 0.001"/>
+			<!-- <mesh filename="~/NASA_ws/digr/description/meshes/wheel_1.stl" scale="0.001 0.001 0.001"/> -->
 			<material name="light_black"/>
 		</visual>
@@ -226,5 +226,5 @@
 	</transmission>
 	<!-- IMU -->
-	<!-- <joint name="imu_joint" type="fixed">
+	<joint name="imu_joint" type="fixed">
 		<axis rpy="0 0 0" xyz="0 1 0"/>
 		<parent link="base_link" />
@@ -246,5 +246,5 @@
 			</geometry>
 		</collision>
-	</link> -->
+	</link>
 <!--PSeye Cameras. One in each top corner -->
 <!--Top right camera -->
@@ -261,4 +261,5 @@
 					<box size="${pseye_camera_length} ${pseye_camera_width} ${pseye_camera_height}"/>
 				</geometry>
+				<material name="red"/>
 			</visual>
 			<collision>
@@ -282,4 +283,5 @@
 			<box size="${pseye_camera_length} ${pseye_camera_width} ${pseye_camera_height}"/>
 		</geometry>
+		<material name="red"/>
 	</visual>
 	<collision>
@@ -303,4 +305,5 @@
 				<box size="${pseye_camera_length} ${pseye_camera_width} ${pseye_camera_height}"/>
 			</geometry>
+			<material name="red"/>
 		</visual>
 		<collision>
@@ -324,4 +327,5 @@
 					<box size="${pseye_camera_length} ${pseye_camera_width} ${pseye_camera_height}"/>
 				</geometry>
+				<material name="red"/>
 			</visual>
 			<collision>

Commit message: bigrdigr_description added drum bigrdigr_gazebo added rough terrian

File: src/bigrdigr_description/urdf/bigrdigr.urdf.xacro (robot description, xacro)
@@ -2,4 +2,22 @@
 <robot name="bigrdigr" xmlns:xacro="https://www.ros.org/wiki/xacro">
 	<xacro:include filename="$(find bigrdigr_description)/urdf/bigrdigr1.gazebo.xacro"/>
+	<material name="grey">
+		<color rgba="0.5 0.5 0.5 1"/>
+	</material>
+	<material name="dark_grey">
+		<color rgba="0.2 0.2 0.2 1"/>
+	</material>
+	<material name="blue">
+		<color rgba="0 0 0.8 1"/>
+	</material>
+	<material name="red">
+		<color rgba="0.8 0 0 1"/>
+	</material>
+	<material name="purple">
+		<color rgba="0.8 0 0.8 1"/>
+	</material>
+	<material name="orange">
+		<color rgba="0.8 0.2 0 1"/>
+	</material>
 	<!-- All units in meters, kg, seconds, rads -->
 	<!-- Equation for inertial matrix of box/prisim -->
@@ -15,4 +33,6 @@
 				 izz="${(m*(3*r*r+h*h))/12.0}"  />
 	</xacro:macro>
+	<!-- Wheel Links -->
+	<xaacro:macro>
 	<!-- Main dimensions: meters, kg, seconds, rads -->
 	<xacro:property name="PI" value="3.1415926535897931" />
@@ -27,4 +47,11 @@
 	<xacro:property name="wheel_height" value="0.15" />
 	<xacro:property name="wheel_mass" value="2.0" />
+	<xacro:property name="arm_length" value="0.4"/>
+	<xacro:property name="arm_height" value="0.06"/>
+	<xacro:property name="arm_width" value="0.06"/>
+	<xacro:property name="arm_mass" value="2.0"/>
+	<xacro:property name="digr_height" value="0.08"/>
+	<xacro:property name="digr_radius" value="0.2"/>
+	<xacro:property name="digr_mass" value="2.0"/>
 	<xacro:property name="imu_length" value="0.025" />
 	<xacro:property name="imu_width" value="0.025" />
@@ -68,18 +95,70 @@
 		</inertial>
 	</link>
-	<joint name="scoop_joint" type="fixed">
-		<parent link="base_link"/>
-		<child link="scoop_link"/>
-		<origin xyz="${base_length/2} 0 ${base_height/2}" rpy="0 0 0"/>
-	</joint>
-	<link name="scoop_link">
+	<joint name="arm_joint" type="fixed">
+		<parent link="base_link"/>
+		<child link="arm_link"/>
+		<origin xyz="${base_length/2+arm_length/2} 0 ${base_height/2}" rpy="0 0 0"/>
+		<dynamics damping="0.5" friction="0.1"/> <!-- get real later-->
+		<limit effort="1000" velocity="10"/> <!-- simmulate motors, max velocity and max joint effort -->
+		<axis xyz="0 1 0"/> <!-- will rotate for y axis -->
+	</joint>
+	<link name="arm_link">
 		<visual>
 			<origin xyz="0 0 0" rpy="0 0 0"/>
 			<geometry>
-				<box size="0.01 0.2 0.2"/>
+				<box size="${arm_length} ${arm_width} ${arm_height}"/>
+			</geometry>
+			<material name="orange"/>
+		</visual>
+		<collision>
+			<origin xyz="0 0 0" rpy="0 0 0"/>
+			<geometry>
+				<box size="${arm_length} ${arm_width} ${arm_height}"/>
+			</geometry>
+		</collision>
+		<inertia>
+			<origin xyz="${arm_length/2} 0 0" rpy="0 0 0"/>
+			<mass value="${arm_mass}"/>
+			<box_inertial_matrix m="${arm_mass}" h="${arm_height}" l="${arm_length}" w="${arm_width}" />
+		</inertia>
+	</link>
+	<joint name="digr_joint" type="continuous">
+		<parent link="arm_link"/>
+		<child link="digr_link"/>
+		<origin xyz="${arm_length/2-0.01} 0 0" rpy="0 0 0"/>
+		<dynamics damping="0.5" friction="0.1"/> <!-- get real later-->
+		<limit effort="1000" velocity="10"/> <!-- simmulate motors, max velocity and max joint effort -->
+		<axis xyz="0 1 0"/> <!-- will rotate for y axis -->
+	</joint>
+	<link name="digr_link">
+		<visual>
+			<origin xyz="0 0 0" rpy="${PI/2.0} 0 0"/>
+			<geometry>
+				<cylinder length="${digr_height}" radius="${digr_radius}" />
 			</geometry>
 			<material name="purple"/>
 		</visual>
-	</link>
+		<collision>
+			<origin xyz="0 0 0" rpy="${PI/2.0} 0 0"/>
+			<geometry>
+				<cylinder length="${digr_height}" radius="${digr_radius}" />
+			</geometry>
+		</collision>
+		<inertia>
+			<origin xyz="0 0 0"/>
+			<mass value="${digr_mass}"/>
+			<cylinder_inertia m="${digr_mass}" h="${digr_height}" r="${digr_radius}"/>
+		</inertia>
+	</link>
+	<!-- <transmission name="digr_trans">
+		<type>transmission_interface/SimpleTransmission</type>
+		<joint name="digr_joint">
+			<hardwareInterface>EffortJointInterface</hardwareInterface>
+		</joint>
+		<actuator name="digr_motor">
+			<hardwareInterface>EffortJointInterface</hardwareInterface>
+			<mechanicalReduction>1</mechanicalReduction>
+		</actuator>
+	</transmission> -->
 	<joint name="front_left_wheel_joint" type="continuous">
 		<parent link="base_link"/>
@@ -252,5 +331,5 @@
 				<box size="${imu_length} ${imu_width} ${imu_height}" />
 			</geometry>
-			<materal name="purple"/>
+			<materal name="blue"/>
 		</visual>
 		<collision>
@@ -337,5 +416,5 @@
 		<link name="pseye_camera4">
 			<visual>
-				<origin xyz="0 0 0" rpy="0 0 0"/>
+				<origin xyz="0 0 0" rpy="0 0 ${PI}"/>
 				<geometry>
 					<box size="${pseye_camera_length} ${pseye_camera_width} ${pseye_camera_height}"/>

File: src/bigrdigr_description/urdf/bigrdigr1.gazebo.xacro (robot description, xacro)
@@ -23,7 +23,18 @@
 		<turnGravityOff>false</turnGravityOff>
 	</gazebo>
-	<gazebo reference="scoop_link">
+	<gazebo reference="arm_link">
+		<material>Gazebo/Orange</material>
+		<mu1>0.3</mu1>
+		<mu2>0.3</mu2>
+	</gazebo>
+	<gazebo reference="digr_link">
 		<material>Gazebo/Purple</material>
-		<turnGravityOff>false</turnGravityOff>
+		<mu1>0.3</mu1>
+		<mu2>0.3</mu2>
+		<kp>1000000.0</kp>
+		<kd>1.0</kd>
+		<minDepth>0.001</minDepth>
+		<maxVel>1</maxVel>
+		<fdir1>1 0 0</fdir1>
 	</gazebo>
 	<gazebo reference="front_left_wheel">
@@ -231,5 +242,5 @@
 			<topic>imu_data</topic>
 			<plugin filename="libgazebo_ros_imu_sensor.so" name="imu_plugin">
-				<topicName>imu</topicName>
+				<topicName>imu/data</topicName>
 				<bodyName>imu_link</bodyName>
 				<updateRateHZ>10.0</updateRateHZ>
@@ -279,6 +290,6 @@
 	    <updateRate>100.0</updateRate>
 	    <robotNamespace>/bigrdigr</robotNamespace>
-			<commandTopic>/cmd_vel</commandTopic>
-			<odometryTopic>/odom</odometryTopic>
+			<commandTopic>cmd_vel</commandTopic>
+			<odometryTopic>odometry/wheel</odometryTopic>
 	    <leftFrontJoint>front_left_wheel_joint</leftFrontJoint>
 	    <rightFrontJoint>front_right_wheel_joint</rightFrontJoint>
