Commit message: bigrdigr/description streamlined code, ros_control working

File: src/bigrdigr_description/urdf/bigrdigr.urdf.xacro (robot description, xacro)
@@ -33,6 +33,4 @@
 				 izz="${(m*(3*r*r+h*h))/12.0}"  />
 	</xacro:macro>
-	<!-- Wheel Links -->
-	<xaacro:macro>
 	<!-- Main dimensions: meters, kg, seconds, rads -->
 	<xacro:property name="PI" value="3.1415926535897931" />

File: src/bigrdigr_description/urdf/bigrdigr_correct.urdf.xacro (robot description, xacro)
@@ -1,4 +1,29 @@
 <?xml version="1.0" encoding="UTF-8"?>
 <robot name="bigrdigr" xmlns:xacro="https://www.ros.org/wiki/xacro">
+  <xacro:include filename="$(find bigrdigr_description)/urdf/wheel.urdf.xacro"/>
+  <xacro:include filename="$(find bigrdigr_description)/urdf/sensors/camera.urdf.xacro"/>
+  <xacro:include filename="$(find bigrdigr_description)/urdf/sensors/imu.urdf.xacro"/>
+  <xacro:include filename="$(find bigrdigr_description)/urdf/extrusion.urdf.xacro"/>
+  <material name="grey">
+    <color rgba="0.5 0.5 0.5 1"/>
+  </material>
+  <material name="dark_grey">
+    <color rgba="0.2 0.2 0.2 1"/>
+  </material>
+  <material name="blue">
+    <color rgba="0 0 0.8 1"/>
+  </material>
+  <material name="red">
+    <color rgba="0.8 0 0 1"/>
+  </material>
+  <material name="green">
+    <color rgba="0 0.5 0 1"/>
+  </material>
+  <material name="purple">
+    <color rgba="0.8 0 0.8 1"/>
+  </material>
+  <material name="orange">
+    <color rgba="0.8 0.2 0 1"/>
+  </material>
   <!-- Hard coded dimenstions well approximating robot -->
   <!-- Robot modeled as:
@@ -9,2 +34,239 @@
        four extensions with cameras, imus, decawaves,
        two rgbd cams front and back center -->
+  <!-- red axis = x axis green axis = y blue axis = z -->
+  <!-- Equation for inertial matrix of box/prisim -->
+  <xacro:macro name="box_inertial_matrix" params="m l w h">
+  	<inertia ixx="${(m*(w*w+h*h))/12.0}" ixy = "0.0" ixz = "0.0"
+     				 iyy="${(m*(l*l+h*h))/12.0}" iyz = "0.0"
+     				 izz="${(m*(l*l+w*w))/12.0}" />
+  </xacro:macro>
+  <!-- Equation for inertial matrix of cylinder (rotating around y axis) -->
+  <xacro:macro name="cylinder_inertia" params="m r h">
+  	<inertia ixx="${(m*(3*r*r+h*h))/12.0}" ixy = "0.0" ixz = "0.0"
+     				 iyy="${m*r*r/2.0}"			   iyz = "0.0"
+     				 izz="${(m*(3*r*r+h*h))/12.0}"  />
+  </xacro:macro>
+  <!-- Main dimensions: meters, kg, seconds, rads -->
+  <xacro:property name="base_height" value="0.54" /> <!--z-->
+	<xacro:property name="base_length" value="0.864925" /> <!--x-->
+	<xacro:property name="base_width" value="0.740" /> <!--y-->
+	<xacro:property name="base_mass" value="72.0" />
+  <xacro:property name="leg_height" value="0.127"/>
+  <xacro:property name="leg_length" value="0.739775"/>
+  <xacro:property name="leg_width" value="0.0508"/>
+  <xacro:property name="leg_mass" value="4"/>
+  <xacro:property name="leg_x_origin_to_axle" value="${leg_length/2-.10835}" />
+	<xacro:property name="leg_y_origin_to_axle" value="0.0254" />
+	<xacro:property name="leg_axle_height" value="0.10535" />
+  <xacro:property name="drum_width" value="${wheel_width/2}"/>
+  <xacro:property name="drum_radius" value="${wheel_radius*1.5}"/>
+  <xacro:property name="drum_mass" value="2"/>
+  <xacro:property name="drum_y_origin_to_base_origin" value="${base_width/4-drum_width/2}"/>
+  <!-- World Origin -->
+	<!-- world_origin is a fictitious link(frame) that is on the ground right below base_link origin -->
+	<!-- z axis is height -->
+	<link name="world_origin"/>
+  <gazebo reference="world_origin">
+		<turnGravityOff>false</turnGravityOff>
+	</gazebo>
+	<joint name="base_footprint_joint" type="fixed">
+		<origin xyz="0 0 ${leg_height-leg_axle_height}" rpy="0 0 0" />
+		<parent link="world_origin" />
+		<child link="base_link" />
+	</joint>
+	<link name="base_link">
+		<visual>
+			<origin xyz="0 0 ${base_height/2.0}" rpy="0 0 0"/>
+			<geometry>
+				<box size=" ${base_length} ${base_width} ${base_height}" />
+			</geometry>
+			<material name="grey"/>
+		</visual>
+		<collision>
+			<origin xyz="0 0 ${base_height/2.0}" rpy="0 0 0"/>
+			<geometry>
+				<box size="${base_length} ${base_width} ${base_width}"/>
+			</geometry>
+		</collision>
+		<inertial>
+			<origin xyz="0 0 ${base_height/2.0}" rpy="0 0 0"/>
+			<mass value="${base_mass}"/>
+			<box_inertial_matrix m="${base_mass}" h="${base_height}" l="${base_length}" w="${base_width}" />
+		</inertial>
+	</link>
+  <gazebo reference="base_link">
+    <material>Gazebo/Grey</material>
+    <turnGravityOff>false</turnGravityOff>
+  </gazebo>
+  <joint name="left_leg_joint" type="fixed">
+		<origin xyz="0 ${base_width/2-leg_width/2} ${-leg_height}" rpy="0 0 0" />
+		<parent link="base_link" />
+		<child link="left_leg" />
+	</joint>
+	<link name="left_leg">
+		<visual>
+			<origin xyz="0 0 ${leg_height/2.0}" rpy="0 0 0"/>
+			<geometry>
+				<box size=" ${leg_length} ${leg_width} ${leg_height}" />
+			</geometry>
+			<material name="grey"/>
+		</visual>
+		<collision>
+			<origin xyz="0 0 ${leg_height/2.0}" rpy="0 0 0"/>
+			<geometry>
+				<box size="${leg_length} ${leg_width} ${leg_width}"/>
+			</geometry>
+		</collision>
+		<inertial>
+			<origin xyz="0 0 ${leg_height/2.0}" rpy="0 0 0"/>
+			<mass value="${leg_mass}"/>
+			<box_inertial_matrix m="${leg_mass}" h="${leg_height}" l="${leg_length}" w="${leg_width}" />
+		</inertial>
+	</link>
+  <gazebo reference="left_leg">
+    <material>Gazebo/Blue</material>
+    <turnGravityOff>false</turnGravityOff>
+  </gazebo>
+  <joint name="right_leg_joint" type="fixed">
+    <origin xyz="0 ${-base_width/2+leg_width/2} ${-leg_height}" rpy="0 0 0" />
+    <parent link="base_link" />
+    <child link="right_leg" />
+  </joint>
+  <link name="right_leg">
+    <visual>
+      <origin xyz="0 0 ${leg_height/2.0}" rpy="0 0 0"/>
+      <geometry>
+        <box size=" ${leg_length} ${leg_width} ${leg_height}" />
+      </geometry>
+      <material name="grey"/>
+    </visual>
+    <collision>
+      <origin xyz="0 0 ${leg_height/2.0}" rpy="0 0 0"/>
+      <geometry>
+        <box size="${leg_length} ${leg_width} ${leg_width}"/>
+      </geometry>
+    </collision>
+    <inertial>
+      <origin xyz="0 0 ${leg_height/2.0}" rpy="0 0 0"/>
+      <mass value="${leg_mass}"/>
+      <box_inertial_matrix m="${leg_mass}" h="${leg_height}" l="${leg_length}" w="${leg_width}" />
+    </inertial>
+  </link>
+  <gazebo reference="right_leg">
+    <material>Gazebo/Blue</material>
+    <turnGravityOff>false</turnGravityOff>
+  </gazebo>
+  <wheel prefix="front_left" leg="left_leg" x="1" y="1"/>
+  <wheel prefix="front_right" leg="right_leg" x="1" y="-1"/>
+  <wheel prefix="back_left" leg="left_leg" x="-1" y="1"/>
+  <wheel prefix="back_right" leg="right_leg" x="-1" y="-1"/>
+  <extrusion prefix="front_left" x="1" y="1"/>
+  <extrusion prefix="front_right" x="1" y="-1"/>
+  <extrusion prefix="back_left" x="-1" y="1"/>
+  <extrusion prefix="back_right" x="-1" y="-1"/>
+  <!-- <camera_macro number="1" x="1" y="1" spin="0"/>
+  <camera_macro number="2" x="1" y="-1" spin="0"/>
+  <camera_macro number="3" x="-1" y="1" spin="${PI}"/>
+  <camera_macro number="4" x="-1" y="-1" spin="${PI}"/> -->
+  <!-- imu and deca front left, back right. in front of extrusion -->
+  <imu number="1"/>
+  <joint name="drum_joint" type="prismatic">
+		<origin xyz="${base_length/2} ${drum_y_origin_to_base_origin} ${base_height/2}" rpy="0 0 0" />
+		<parent link="base_link" />
+		<child link="drum" />
+    <axis xyz="0 0 1"/>
+    <dynamics damping="0.1" friction="0.1"/> <!-- get real Ns/m damping N friction -->
+    <limit lower="${-base_length/2}" upper="${base_length/2}" effort="1000" velocity="10"/> <!-- m distance, max effort and vel -->
+	</joint>
+	<link name="drum">
+		<visual>
+			<origin xyz="0 ${drum_width/2} 0" rpy="${PI/2.0} 0 0"/>
+			<geometry>
+				<cylinder length="${drum_width}" radius="${drum_radius}" />
+			</geometry>
+			<material name="purple"/>
+		</visual>
+		<collision>
+			<origin xyz="0 ${drum_width/2} 0" rpy="${PI/2.0} 0 0"/>
+			<geometry>
+				<cylinder length="${drum_width}" radius="${drum_radius}" />
+			</geometry>
+		</collision>
+		<inertial>
+			<origin xyz="${drum_radius/2} ${drum_width/2} 0" rpy="${PI/2.0} 0 0"/>
+			<mass value="${leg_mass}"/>
+			<cylinder_inertia m="${drum_mass}" r="${drum_radius}" h="${drum_width}"/>
+		</inertial>
+	</link>
+  <transmission name="drum_trans">
+    <type>transmission_interface/SimpleTransmission</type>
+    <joint name="drum_joint">
+      <hardwareInterface>hardware_interface/PositionJointInterface</hardwareInterface>
+    </joint>
+    <actuator name="drum_motor">
+      <hardwareInterface>hardware_interface/PositionJointInterface</hardwareInterface>
+      <mechanicalReduction>1</mechanicalReduction>
+    </actuator>
+  </transmission>
+  <gazebo reference="drum">
+    <material>Gazebo/Purple</material>
+    <turnGravityOff>false</turnGravityOff>
+  </gazebo>
+  <!-- <gazebo>
+	  <plugin name="differential_drive_controller1" filename="libgazebo_ros_diff_drive.so">
+	    <alwaysOn>true</alwaysOn>
+	    <updateRate>100</updateRate>
+	    <leftJoint>front_left_wheel_joint</leftJoint>
+	    <rightJoint>front_right_wheel_joint</rightJoint>
+	    <wheelSeparation>${2*base_x_origin_to_wheel_origin}</wheelSeparation>
+	    <wheelDiameter>${2*wheel_radius}</wheelDiameter>
+	    <torque>20</torque>
+	    <commandTopic>cmd_vel</commandTopic>
+	    <odometryTopic>odom</odometryTopic>
+	    <odometryFrame>odom</odometryFrame>
+	    <robotBaseFrame>world_origin</robotBaseFrame>
+			<legacyMode>false</legacyMode>
+	  </plugin>
+	</gazebo>
+	<gazebo>
+	  <plugin name="differential_drive_controller2" filename="libgazebo_ros_diff_drive.so">
+	    <alwaysOn>true</alwaysOn>
+	    <updateRate>100</updateRate>
+	    <leftJoint>back_left_wheel_joint</leftJoint>
+	    <rightJoint>back_right_wheel_joint</rightJoint>
+	    <wheelSeparation>${2*base_x_origin_to_wheel_origin}</wheelSeparation>
+	    <wheelDiameter>${2*wheel_radius}</wheelDiameter>
+	    <torque>20</torque>
+	    <commandTopic>cmd_vel</commandTopic>
+	    <odometryTopic>odom</odometryTopic>
+	    <odometryFrame>odom</odometryFrame>
+	    <robotBaseFrame>world_origin</robotBaseFrame>
+			<legacyMode>false</legacyMode>
+	  </plugin>
+	</gazebo> -->
+	<gazebo>
+	  <plugin name="skid_steer_drive_controller" filename="libgazebo_ros_skid_steer_drive.so">
+	    <updateRate>100.0</updateRate>
+	    <robotNamespace>/bigrdigr</robotNamespace>
+			<commandTopic>cmd_vel</commandTopic>
+			<odometryTopic>odometry/wheel</odometryTopic>
+	    <leftFrontJoint>front_left_wheel_joint</leftFrontJoint>
+	    <rightFrontJoint>front_right_wheel_joint</rightFrontJoint>
+	    <leftRearJoint>back_left_wheel_joint</leftRearJoint>
+	    <rightRearJoint>back_right_wheel_joint</rightRearJoint>
+	    <wheelSeparation>${2*base_width}</wheelSeparation>
+	    <wheelDiameter>${2*wheel_radius}</wheelDiameter>
+	    <robotBaseFrame>base_link</robotBaseFrame>
+	    <torque>20</torque>
+	    <broadcastTF>true</broadcastTF>
+			<legacyMode>false</legacyMode>
+	  </plugin>
+	</gazebo>
+  <gazebo>
+  <plugin name="gazebo_ros_control" filename="libgazebo_ros_control.so">
+    <robotNamespace>/bigrdigr</robotNamespace>
+    <robotSimType>gazebo_ros_control/DefaultRobotHWSim</robotSimType>
+    <legacyMode>false</legacyMode>
+  </plugin>
+</gazebo>
+</robot>

File: src/bigrdigr_description/urdf/sensors/camera.urdf.xacro (robot description, xacro)
@@ -1,26 +1,78 @@
 <?xml version="1.0" ?>
-<xacro:macro name="camera_joint" params="camera_name">
-  <joint name="${camera_name}_camera_joint" type="fixed">
-    <axis xyz="0 1 0" />
-    <origin xyz="${base_width/2} ${-base_length/2.0} ${base_height}" rpy="0 0 0"/>
-    <parent link="base_link"/>
-    <child link="${camera_name}"/>
-  </joint>
-</xacro:macro>
-<xacro:macro name="camera" params="camera_name">
-  <link name="pseye_camera3">
-    <visual>
-      <origin xyz="0 0 0" rpy="0 0 0"/>
-      <geometry>
-        <box size="${pseye_camera_length} ${pseye_camera_width} ${pseye_camera_height}"/>
-      </geometry>
-      <material name="red"/>
-    </visual>
-    <collision>
-      <origin xyz="0 0 0" rpy="0 0 0" />
-      <geometry>
-        <box size="${pseye_camera_length} ${pseye_camera_width} ${pseye_camera_height}"/>
-      </geometry>
-    </collision>
-  </link>
-</xacro:macro>
+<robot name="bigrdigr" xmlns:xacro="https://www.ros.org/wiki/xacro">
+  <!-- Main dimensions: meters, kg, seconds, rads -->
+  <xacro:property name="pseye_camera_height" value="0.08" />
+	<xacro:property name="pseye_camera_length" value="0.07" />
+	<xacro:property name="pseye_camera_width" value="0.09" />
+  <xacro:property name="pseye_FOV" value="1.309"/> <!--56 or 75 degrees, need rad-->
+  <xacro:macro name="camera_link" params="number">
+    <link name="pseye_camera${number}">
+      <visual>
+        <origin xyz="0 0 0" rpy="0 0 0"/>
+        <geometry>
+          <box size="${pseye_camera_length} ${pseye_camera_width} ${pseye_camera_height}"/>
+        </geometry>
+        <material name="red"/>
+      </visual>
+      <collision>
+        <origin xyz="0 0 0" rpy="0 0 0" />
+        <geometry>
+          <box size="${pseye_camera_length} ${pseye_camera_width} ${pseye_camera_height}"/>
+        </geometry>
+      </collision>
+    </link>
+  </xacro:macro>
+  <xacro:macro name="camera_joint" params="number x y spin">
+    <joint name="camera${number}_joint" type="fixed">
+      <origin xyz="${x*(base_length/2-pseye_camera_length/2)} ${y*(base_width/2+pseye_camera_width/2)} ${base_height-pseye_camera_height/2}" rpy="0 0 ${spin}"/>
+      <parent link="base_link"/>
+      <child link="pseye_camera${number}"/>
+    </joint>
+  </xacro:macro>
+  <xacro:macro name="camera_gazebo" params="number">
+    <gazebo reference="pseye_camera${number}">
+  		<material>Gazebo/Red</material>
+  		<sensor type="camera" name="cam${number}">
+  			<update_rate>120</update_rate> <!--fps? -->
+  			<camera name="camera${number}">
+  				<horizontal_fov>${pseye_FOV}</horizontal_fov>
+  				<image>
+  					<width>320</width>
+  					<height>240</height>
+  					<format>R8G8B8</format>
+  				</image>
+  				<clip> <!--distance (m) limits on where a camera can see an object need to find -->
+  					<near>0.02</near>
+  					<far>300</far>
+  				</clip>
+  				<noise>
+  					<type>gaussian</type>
+  					<mean>0.0</mean>
+  					<stddev>0.007</stddev>
+  				</noise>
+  			</camera>
+  			<plugin name="camera_controller" filename="libgazebo_ros_camera.so">
+  				<alwaysOn>true</alwaysOn>
+  				<!--Nodes-->
+  				<updateRate>0.0</updateRate>
+  				<cameraName>camera/pseye_camera${number}</cameraName>
+  				<imageTopicName>image_raw</imageTopicName>
+  				<cameraInfoTopicName>camera_info</cameraInfoTopicName>
+  				<frameName>pseye_camera${number}</frameName>
+  				<!--May need to find? -->
+  				<hackBaseline>0.07</hackBaseline>
+  				<distortionK1>0.0</distortionK1>
+  				<distortionK2>0.0</distortionK2>
+  				<distortionK3>0.0</distortionK3>
+  				<distortionT1>0.0</distortionT1>
+  				<distortionT2>0.0</distortionT2>
+  			</plugin>
+  		</sensor>
+  	</gazebo>
+  </xacro:macro>
+  <xacro:macro name="camera_macro" params="number x y spin">
+    <camera_link number="${number}"/>
+    <camera_joint number="${number}" x="${x}" y="${y}" spin="${spin}"/>
+    <camera_gazebo number="${number}"/>
+  </xacro:macro>
+</robot>

File: src/bigrdigr_description/urdf/wheel.urdf.xacro (robot description, xacro)
@@ -1,25 +1,25 @@
 <?xml version="1.0" ?>
 <robot name="bigrdigr" xmlns:xacro="https://www.ros.org/wiki/xacro">
-	<xacro:property name="PI" value="3.141592653589793238462643383279502884197" />
 	<!--here are a lot of the measurements. currently, all of them are just dummy values.
 	change these later when it will be useful to do so.-->
-	<xacro:property name="wheel_height" value="1" />
-	<xacro:property name="wheel_radius" value="1" />
-	<xacro:property name="wheel_mass" value="1" />
+	<!-- Main dimensions: meters, kg, seconds, rads -->
+	<xacro:property name="PI" value="3.141592653589793238462643383279502884197" />
+	<xacro:property name="wheel_width" value=".15" />
+	<xacro:property name="wheel_radius" value=".18035" />
+	<xacro:property name="wheel_mass" value="2" />
 	<!--here is a macro for a wheel -->
-	<xacro:macro name="wheel" params="prefix">
+	<xacro:macro name="wheel_link" params="prefix">
 		<link name="${prefix}_wheel">
 			<visual>
 				<origin xyz="0 0 0" rpy="${PI/2.0} 0 0"/>
 	      <geometry>
-          <cylinder length="${wheel_height}" radius="${wheel_radius}" />
+          <cylinder length="${wheel_width}" radius="${wheel_radius}" />
         </geometry>
-        <!-- <mesh filename="~/NASA_ws/digr/description/meshes/wheel_1.stl" scale="0.001 0.001 0.001"/> -->
         <material name="light_black"/>
-			<\visual>
+			</visual>
 	    <collision>
         <origin xyz="0 0 0" rpy="${PI/2.0} 0 0" />
         <geometry>
-          <cylinder length="${wheel_height}" radius="${wheel_radius}" />
+          <cylinder length="${wheel_width}" radius="${wheel_radius}" />
        	</geometry>
 	    </collision>
@@ -27,17 +27,29 @@
        	<origin xyz="0 0 0" />
       	<mass value="${wheel_mass}" />
-       	<cylinder_inertia m="${wheel_mass}" h="${wheel_height}" r="${wheel_radius}"/>
+       	<cylinder_inertia m="${wheel_mass}" h="${wheel_width}" r="${wheel_radius}"/>
       </inertial>
 		</link>
 	</xacro:macro>
-	<xacro:macro name="wheel_joint" params="prefix">
+	<xacro:macro name="wheel_joint" params="prefix leg x y">
 		<joint name="${prefix}_wheel_joint" type="continuous">
-			<parent link="base_link" />
+			<parent link="${leg}" />
 			<child 	link="${prefix}_wheel" />
-      <origin xyz="${base_x_origin_to_wheel_origin} ${base_y_origin_to_wheel_origin} 0" rpy="0 0 0"/>
-      <dynamics damping="0.5" friction="0.1"/> <!-- get real later-->
+      <origin xyz="${x*leg_x_origin_to_axle} ${y*(wheel_radius/2+leg_width/4)} ${leg_axle_height-leg_height/2}" rpy="0 0 0"/>
+      <dynamics damping="0.5" friction="0.1"/> <!-- get real later N*m*s/rad damp N*m friction-->
       <limit effort="1000" velocity="10"/> <!-- simmulate motors, max velocity and max joint effort -->
       <axis xyz="0 1 0"/> <!-- will rotate for y axis -->
     </joint>
+	</xacro:macro>
+	<xacro:macro name="wheel_gazebo" params="prefix">
+		<gazebo reference="${prefix}_wheel">
+			<mu1>0.3</mu1>
+			<mu2>0.3</mu2>
+			<kp>1000000.0</kp>
+			<kd>1.0</kd>
+			<minDepth>0.001</minDepth>
+			<maxVel>1</maxVel>
+			<fdir1>1 0 0</fdir1>
+			<material>Gazebo/FlatBlack</material>
+		</gazebo>
 	</xacro:macro>
   <xacro:macro name="wheel_trans" params="prefix">
@@ -45,5 +57,5 @@
       <type>transmission_interface/SimpleTransmission</type>
       <joint name="${prefix}_wheel_joint">
-        <hardwareInterface>EffortJointInterface</hardwareInterface>
+        <hardwareInterface>hardware_interface/EffortJointInterface</hardwareInterface>
       </joint>
       <actuator name="${prefix}_wheel_motor">
@@ -53,3 +65,9 @@
     </transmission>
   </xacro:macro>
+	<xacro:macro name="wheel" params="prefix leg x y">
+		<wheel_link prefix="${prefix}"/>
+		<wheel_joint prefix="${prefix}" leg="${leg}" x="${x}" y="${y}"/>
+		<wheel_gazebo prefix="${prefix}"/>
+		<wheel_trans prefix="${prefix}"/>
+	</xacro:macro>
 </robot>
