Commit message: bigrdigr_description bigrdigr_gazebo streamlined file names, added arg for cameras and paused

File: src/bigrdigr_description/urdf/bigrdigr.urdf.xacro (robot description, xacro)
@@ -1,72 +1,76 @@
-<?xml version="1.0" ?>
+<?xml version="1.0" encoding="UTF-8"?>
 <robot name="bigrdigr" xmlns:xacro="https://www.ros.org/wiki/xacro">
-	<xacro:include filename="$(find bigrdigr_description)/urdf/bigrdigr1.gazebo.xacro"/>
-	<material name="grey">
-		<color rgba="0.5 0.5 0.5 1"/>
-	</material>
-	<material name="dark_grey">
-		<color rgba="0.2 0.2 0.2 1"/>
-	</material>
-	<material name="blue">
-		<color rgba="0 0 0.8 1"/>
-	</material>
-	<material name="red">
-		<color rgba="0.8 0 0 1"/>
-	</material>
-	<material name="purple">
-		<color rgba="0.8 0 0.8 1"/>
-	</material>
-	<material name="orange">
-		<color rgba="0.8 0.2 0 1"/>
-	</material>
-	<!-- All units in meters, kg, seconds, rads -->
-	<!-- Equation for inertial matrix of box/prisim -->
-	<xacro:macro name="box_inertial_matrix" params="m l w h">
-		<inertia ixx="${(m*(w*w+h*h))/12.0}" ixy = "0.0" ixz = "0.0"
-				 iyy="${(m*(l*l+h*h))/12.0}" iyz = "0.0"
-				 izz="${(m*(l*l+w*w))/12.0}" />
-	</xacro:macro>
-	<!-- Equation for inertial matrix of cylinder (rotating around y axis) -->
-	<xacro:macro name="cylinder_inertia" params="m r h">
-		<inertia ixx="${(m*(3*r*r+h*h))/12.0}" ixy = "0.0" ixz = "0.0"
-				 iyy="${m*r*r/2.0}"			   iyz = "0.0"
-				 izz="${(m*(3*r*r+h*h))/12.0}"  />
-	</xacro:macro>
-	<!-- Main dimensions: meters, kg, seconds, rads -->
-	<xacro:property name="PI" value="3.1415926535897931" />
-	<xacro:property name="base_height" value="0.690" />
-	<xacro:property name="base_length" value="0.740" />
-	<xacro:property name="base_width" value="0.865" />
+  <xacro:include filename="$(find bigrdigr_description)/urdf/wheel.urdf.xacro"/>
+  <xacro:include filename="$(find bigrdigr_description)/urdf/sensors/camera.urdf.xacro"/>
+  <xacro:include filename="$(find bigrdigr_description)/urdf/sensors/imu.urdf.xacro"/>
+  <xacro:include filename="$(find bigrdigr_description)/urdf/extrusion.urdf.xacro"/>
+  <material name="grey">
+    <color rgba="0.5 0.5 0.5 1"/>
+  </material>
+  <material name="dark_grey">
+    <color rgba="0.2 0.2 0.2 1"/>
+  </material>
+  <material name="blue">
+    <color rgba="0 0 0.8 1"/>
+  </material>
+  <material name="red">
+    <color rgba="0.8 0 0 1"/>
+  </material>
+  <material name="green">
+    <color rgba="0 0.5 0 1"/>
+  </material>
+  <material name="purple">
+    <color rgba="0.8 0 0.8 1"/>
+  </material>
+  <material name="orange">
+    <color rgba="0.8 0.2 0 1"/>
+  </material>
+  <!-- Hard coded dimenstions well approximating robot -->
+  <!-- Robot modeled as:
+       a large box (base_link), origin at bottom,
+       two base_legs, beneath it,
+       four wheels, two on each base_leg,
+       a box that reps the drum,
+       four extensions with cameras, imus, decawaves,
+       two rgbd cams front and back center -->
+  <!-- red axis = x axis green axis = y blue axis = z -->
+  <!-- Equation for inertial matrix of box/prisim -->
+  <xacro:macro name="box_inertial_matrix" params="m l w h">
+  	<inertia ixx="${(m*(w*w+h*h))/12.0}" ixy = "0.0" ixz = "0.0"
+     				 iyy="${(m*(l*l+h*h))/12.0}" iyz = "0.0"
+     				 izz="${(m*(l*l+w*w))/12.0}" />
+  </xacro:macro>
+  <!-- Equation for inertial matrix of cylinder (rotating around y axis) -->
+  <xacro:macro name="cylinder_inertia" params="m r h">
+  	<inertia ixx="${(m*(3*r*r+h*h))/12.0}" ixy = "0.0" ixz = "0.0"
+     				 iyy="${m*r*r/2.0}"			   iyz = "0.0"
+     				 izz="${(m*(3*r*r+h*h))/12.0}"  />
+  </xacro:macro>
+  <!-- Main dimensions: meters, kg, seconds, rads -->
+  <xacro:property name="base_height" value="0.54" /> <!--z-->
+	<xacro:property name="base_length" value="0.864925" /> <!--x-->
+	<xacro:property name="base_width" value="0.740" /> <!--y-->
 	<xacro:property name="base_mass" value="72.0" />
-	<xacro:property name="base_x_origin_to_wheel_origin" value="0.29125" />
-	<xacro:property name="base_y_origin_to_wheel_origin" value="0.190" />
-	<xacro:property name="base_height_origin_to_wheel_origin" value="0.103" />
-	<xacro:property name="wheel_radius" value="0.174" />
-	<xacro:property name="wheel_height" value="0.15" />
-	<xacro:property name="wheel_mass" value="2.0" />
-	<xacro:property name="arm_length" value="0.4"/>
-	<xacro:property name="arm_height" value="0.06"/>
-	<xacro:property name="arm_width" value="0.06"/>
-	<xacro:property name="arm_mass" value="2.0"/>
-	<xacro:property name="digr_height" value="0.08"/>
-	<xacro:property name="digr_radius" value="0.2"/>
-	<xacro:property name="digr_mass" value="2.0"/>
-	<xacro:property name="imu_length" value="0.025" />
-	<xacro:property name="imu_width" value="0.025" />
-	<xacro:property name="imu_height" value="0.01" />
-	<xacro:property name="pseye_camera_height" value="0.08" />
-	<xacro:property name="pseye_camera_length" value="0.07" />
-	<xacro:property name="pseye_camera_width" value="0.09" />
-	<!-- 4 top corners-->
-	<!--<xacro:property name="realSense_camera_height" value="0.09" />
-	<xacro:property name="realSense_camera_length" value="0.025" />
-	<xacro:property name="realSense_camera_width" value="0.025" />-->
- <!--front middle-in, back middle-in, top middle -->
-	<!-- World Origin -->
+  <xacro:property name="leg_height" value="0.127"/>
+  <xacro:property name="leg_length" value="0.739775"/>
+  <xacro:property name="leg_width" value="0.0508"/>
+  <xacro:property name="leg_mass" value="4"/>
+  <xacro:property name="leg_x_origin_to_axle" value="${leg_length/2-.10835}" />
+	<xacro:property name="leg_y_origin_to_axle" value="0.0254" />
+	<xacro:property name="leg_axle_height" value="0.10535" />
+  <xacro:property name="drum_height" value=".11809"/>
+  <xacro:property name="drum_length" value="${base_length+.01}"/>
+  <xacro:property name="drum_width" value=".34"/>
+  <xacro:property name="drum_mass" value="2"/>
+  <xacro:property name="drum_y_origin_to_base_origin" value="${base_width/2-drum_width/2}"/>
+  <!-- World Origin -->
 	<!-- world_origin is a fictitious link(frame) that is on the ground right below base_link origin -->
 	<!-- z axis is height -->
 	<link name="world_origin"/>
+  <gazebo reference="world_origin">
+		<turnGravityOff>false</turnGravityOff>
+	</gazebo>
 	<joint name="base_footprint_joint" type="fixed">
-		<origin xyz="0 0 ${wheel_radius - base_height_origin_to_wheel_origin}" rpy="0 0 0" />
+		<origin xyz="0 0 ${leg_height-leg_axle_height}" rpy="0 0 0" />
 		<parent link="world_origin" />
 		<child link="base_link" />
@@ -77,5 +81,4 @@
 			<geometry>
 				<box size=" ${base_length} ${base_width} ${base_height}" />
-				<!-- <mesh filename="~/NASA_ws/digr/description/meshes/base_link.stl" scale="0.001 0.001 0.001"/> -->
 			</geometry>
 			<material name="grey"/>
@@ -93,338 +96,184 @@
 		</inertial>
 	</link>
-	<joint name="arm_joint" type="fixed">
-		<parent link="base_link"/>
-		<child link="arm_link"/>
-		<origin xyz="${base_length/2+arm_length/2} 0 ${base_height/2}" rpy="0 0 0"/>
-		<dynamics damping="0.5" friction="0.1"/> <!-- get real later-->
-		<limit effort="1000" velocity="10"/> <!-- simmulate motors, max velocity and max joint effort -->
-		<axis xyz="0 1 0"/> <!-- will rotate for y axis -->
+  <gazebo reference="base_link">
+    <material>Gazebo/Grey</material>
+    <turnGravityOff>false</turnGravityOff>
+  </gazebo>
+  <joint name="left_leg_joint" type="fixed">
+		<origin xyz="0 ${base_width/2-leg_width/2} ${-leg_height}" rpy="0 0 0" />
+		<parent link="base_link" />
+		<child link="left_leg" />
 	</joint>
-	<link name="arm_link">
+	<link name="left_leg">
 		<visual>
-			<origin xyz="0 0 0" rpy="0 0 0"/>
-			<geometry>
-				<box size="${arm_length} ${arm_width} ${arm_height}"/>
-			</geometry>
-			<material name="orange"/>
+			<origin xyz="0 0 ${leg_height/2.0}" rpy="0 0 0"/>
+			<geometry>
+				<box size=" ${leg_length} ${leg_width} ${leg_height}" />
+			</geometry>
+			<material name="blue"/>
 		</visual>
 		<collision>
-			<origin xyz="0 0 0" rpy="0 0 0"/>
-			<geometry>
-				<box size="${arm_length} ${arm_width} ${arm_height}"/>
-			</geometry>
-		</collision>
-		<inertia>
-			<origin xyz="${arm_length/2} 0 0" rpy="0 0 0"/>
-			<mass value="${arm_mass}"/>
-			<box_inertial_matrix m="${arm_mass}" h="${arm_height}" l="${arm_length}" w="${arm_width}" />
-		</inertia>
-	</link>
-	<joint name="digr_joint" type="continuous">
-		<parent link="arm_link"/>
-		<child link="digr_link"/>
-		<origin xyz="${arm_length/2-0.01} 0 0" rpy="0 0 0"/>
-		<dynamics damping="0.5" friction="0.1"/> <!-- get real later-->
-		<limit effort="1000" velocity="10"/> <!-- simmulate motors, max velocity and max joint effort -->
-		<axis xyz="0 1 0"/> <!-- will rotate for y axis -->
-	</joint>
-	<link name="digr_link">
-		<visual>
-			<origin xyz="0 0 0" rpy="${PI/2.0} 0 0"/>
-			<geometry>
-				<cylinder length="${digr_height}" radius="${digr_radius}" />
-			</geometry>
-			<material name="purple"/>
-		</visual>
-		<collision>
-			<origin xyz="0 0 0" rpy="${PI/2.0} 0 0"/>
-			<geometry>
-				<cylinder length="${digr_height}" radius="${digr_radius}" />
-			</geometry>
-		</collision>
-		<inertia>
-			<origin xyz="0 0 0"/>
-			<mass value="${digr_mass}"/>
-			<cylinder_inertia m="${digr_mass}" h="${digr_height}" r="${digr_radius}"/>
-		</inertia>
-	</link>
-	<!-- <transmission name="digr_trans">
-		<type>transmission_interface/SimpleTransmission</type>
-		<joint name="digr_joint">
-			<hardwareInterface>EffortJointInterface</hardwareInterface>
-		</joint>
-		<actuator name="digr_motor">
-			<hardwareInterface>EffortJointInterface</hardwareInterface>
-			<mechanicalReduction>1</mechanicalReduction>
-		</actuator>
-	</transmission> -->
-	<joint name="front_left_wheel_joint" type="continuous">
-		<parent link="base_link"/>
-		<child link="front_left_wheel"/>
-		<origin xyz="${base_x_origin_to_wheel_origin} ${base_y_origin_to_wheel_origin} 0" rpy="0 0 0"/>
-		<dynamics damping="0.5" friction="0.1"/> <!-- get real later-->
-		<limit effort="1000" velocity="10"/> <!-- simmulate motors, max velocity and max joint effort -->
-		<axis xyz="0 1 0"/> <!-- will rotate for y axis -->
-	</joint>
-	<link name="front_left_wheel">
-		<visual>
-			<origin xyz="0 0 0" rpy="${PI/2.0} 0 0"/>
-			<geometry>
-				<cylinder length="${wheel_height}" radius="${wheel_radius}" />
-			</geometry>
-			<!-- <mesh filename="~/NASA_ws/digr/description/meshes/wheel_1.stl" scale="0.001 0.001 0.001"/> -->
-			<material name="light_black"/>
-		</visual>
-		<collision>
-			<origin xyz="0 0 0" rpy="${PI/2.0} 0 0" />
-			<geometry>
-				<cylinder length="${wheel_height}" radius="${wheel_radius}" />
+			<origin xyz="0 0 ${leg_height/2.0}" rpy="0 0 0"/>
+			<geometry>
+				<box size="${leg_length} ${leg_width} ${leg_width}"/>
 			</geometry>
 		</collision>
 		<inertial>
-			<origin xyz="0 0 0" />
-			<mass value="${wheel_mass}" />
-			<cylinder_inertia m="${wheel_mass}" h="${wheel_height}" r="${wheel_radius}"/>
+			<origin xyz="0 0 ${leg_height/2.0}" rpy="0 0 0"/>
+			<mass value="${leg_mass}"/>
+			<box_inertial_matrix m="${leg_mass}" h="${leg_height}" l="${leg_length}" w="${leg_width}" />
 		</inertial>
 	</link>
-	<transmission name="front_left_wheel_trans">
-		<type>transmission_interface/SimpleTransmission</type>
-		<joint name="front_left_wheel_joint">
-			<hardwareInterface>EffortJointInterface</hardwareInterface>
-		</joint>
-		<actuator name="front_left_wheel_motor">
-			<hardwareInterface>EffortJointInterface</hardwareInterface>
-			<mechanicalReduction>1</mechanicalReduction>
-		</actuator>
-	</transmission>
-	<!-- Transmission sims motor control -->
-	<joint name="front_right_wheel_joint" type="continuous">
-		<parent link="base_link"/>
-		<child link="front_right_wheel"/>
-		<origin xyz="${base_x_origin_to_wheel_origin} ${-base_y_origin_to_wheel_origin} 0" rpy="0 0 0"/>
-		<dynamics damping="0.5" friction="0.1"/> <!-- get real later-->
-		<limit effort="1000" velocity="10"/> <!-- simmulate motors, max velocity and max joint effort -->
-		<axis xyz="0 1 0"/> <!-- will rotate for y axis -->
+  <gazebo reference="left_leg">
+    <material>Gazebo/Blue</material>
+    <turnGravityOff>false</turnGravityOff>
+  </gazebo>
+  <joint name="right_leg_joint" type="fixed">
+    <origin xyz="0 ${-base_width/2+leg_width/2} ${-leg_height}" rpy="0 0 0" />
+    <parent link="base_link" />
+    <child link="right_leg" />
+  </joint>
+  <link name="right_leg">
+    <visual>
+      <origin xyz="0 0 ${leg_height/2.0}" rpy="0 0 0"/>
+      <geometry>
+        <box size=" ${leg_length} ${leg_width} ${leg_height}" />
+      </geometry>
+      <material name="blue"/>
+    </visual>
+    <collision>
+      <origin xyz="0 0 ${leg_height/2.0}" rpy="0 0 0"/>
+      <geometry>
+        <box size="${leg_length} ${leg_width} ${leg_width}"/>
+      </geometry>
+    </collision>
+    <inertial>
+      <origin xyz="0 0 ${leg_height/2.0}" rpy="0 0 0"/>
+      <mass value="${leg_mass}"/>
+      <box_inertial_matrix m="${leg_mass}" h="${leg_height}" l="${leg_length}" w="${leg_width}" />
+    </inertial>
+  </link>
+  <gazebo reference="right_leg">
+    <material>Gazebo/Blue</material>
+    <turnGravityOff>false</turnGravityOff>
+  </gazebo>
+  <wheel prefix="front_left" leg="left_leg" x="1" y="1"/>
+  <wheel prefix="front_right" leg="right_leg" x="1" y="-1"/>
+  <wheel prefix="back_left" leg="left_leg" x="-1" y="1"/>
+  <wheel prefix="back_right" leg="right_leg" x="-1" y="-1"/>
+  <extrusion prefix="front_left" x="1" y="1"/>
+  <extrusion prefix="front_right" x="1" y="-1"/>
+  <extrusion prefix="back_left" x="-1" y="1"/>
+  <extrusion prefix="back_right" x="-1" y="-1"/>
+  <!-- cameras under extrusions -->
+  <xacro:arg name="cameras" default="false"/>
+  <xacro:property name="useCams" value="$(arg cameras)"/>
+  <xacro:if value="${useCams == 'true'}">
+    <camera_macro number="1" y="1" extrusion="front_left_extrusion" spin="0"/>
+    <camera_macro number="2" y="-1" extrusion="front_right_extrusion" spin="0"/>
+    <camera_macro number="3" y="1" extrusion="back_left_extrusion" spin="${PI}"/>
+    <camera_macro number="4" y="-1" extrusion="back_right_extrusion" spin="${PI}"/>
+  </xacro:if>
+  <!-- imu and deca front left, back right. in front of extrusion -->
+  <imu number="1" x="1" y="1" extrusion="front_left_extrusion"/>
+  <imu number="2" x="1" y="-1" extrusion="back_right_extrusion"/>
+  <joint name="drum_joint" type="prismatic">
+		<origin xyz="0 ${drum_y_origin_to_base_origin} ${-drum_height/2}" rpy="0 0 0" />
+		<parent link="base_link" />
+		<child link="drum" />
+    <axis xyz="0 0 1"/>
+    <dynamics damping="0.1" friction="0.1"/> <!-- get real Ns/m damping N friction -->
+    <limit lower="0" upper="${base_height}" effort="1000" velocity="10"/> <!-- m distance, max effort and vel -->
 	</joint>
-	<link name="front_right_wheel">
-		<visual>
-			<origin xyz="0 0 0" rpy="${PI/2.0} 0 0"/>
-			<geometry>
-				<cylinder length="${wheel_height}" radius="${wheel_radius}" />
-			</geometry>
-			<!-- <mesh filename="~/NASA_ws/digr/description/meshes/wheel_1.stl" scale="0.001 0.001 0.001"/> -->
-			<material name="light_black"/>
-		</visual>
-		<collision>
-			<origin xyz="0 0 0" rpy="${PI/2.0} 0 0" />
-			<geometry>
-				<cylinder length="${wheel_height}" radius="${wheel_radius}" />
-			</geometry>
-		</collision>
-		<inertial>
-			<origin xyz="0 0 0" />
-			<mass value="${wheel_mass}" />
-			<cylinder_inertia m="${wheel_mass}" h="${wheel_height}" r="${wheel_radius}"/>
-		</inertial>
+	<link name="drum">
+    <visual>
+      <origin xyz="0 0 0" rpy="0 0 0"/>
+      <geometry>
+        <box size=" ${drum_length} ${drum_width} ${drum_height}" />
+      </geometry>
+      <material name="purple"/>
+    </visual>
+    <collision>
+      <origin xyz="0 0 0" rpy="0 0 0"/>
+      <geometry>
+        <box size="${drum_length} ${drum_width} ${drum_width}"/>
+      </geometry>
+    </collision>
+    <inertial>
+      <origin xyz="0 0 0" rpy="0 0 0"/>
+      <mass value="${drum_mass}"/>
+      <box_inertial_matrix m="${drum_mass}" h="${drum_height}" l="${drum_length}" w="${drum_width}" />
+    </inertial>
 	</link>
-	<transmission name="front_left_wheel_trans">
-		<type>transmission_interface/SimpleTransmission</type>
-		<joint name="front_left_wheel_joint">
-			<hardwareInterface>EffortJointInterface</hardwareInterface>
-		</joint>
-		<actuator name="front_left_wheel_motor">
-			<hardwareInterface>EffortJointInterface</hardwareInterface>
-			<mechanicalReduction>1</mechanicalReduction>
-		</actuator>
-	</transmission>
-	<joint name="back_left_wheel_joint" type="continuous">
-		<parent link="base_link"/>
-		<child link="back_left_wheel"/>
-		<origin xyz="${-base_x_origin_to_wheel_origin} ${base_y_origin_to_wheel_origin} 0" rpy="0 0 0"/>
-		<dynamics damping="0.5" friction="0.1"/> <!-- get real later-->
-		<limit effort="1000" velocity="10"/> <!-- simmulate motors, max velocity and max joint effort -->
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
File: src/bigrdigr_description/urdf/extrusion.urdf.xacro (robot description, xacro)
@@ -3,10 +3,11 @@
   <!-- Main dimensions: meters, kg, seconds, rads -->
   <xacro:property name="extrusion_height" value="0.0254"/>
-  <xacro:property name="extrusion_length" value="0.0946"/>
+  <xacro:property name="extrusion_length" value="0.0254"/>
   <xacro:property name="extrusion_width" value="0.13254"/>
   <xacro:property name="extrusion_mass" value="0.5"/>
+  <xacro:property name="extrusion_edge_to_base_edge" value="0.0946"/>
   <xacro:macro name="extrusion_joint" params="prefix x y">
     <joint name="${prefix}_extrusion_joint" type="fixed">
-      <origin xyz="${x*(base_length/2-extrusion_length/2)} ${y*base_width/2} ${base_height-extrusion_height/2}" rpy="0 0 0"/>
+      <origin xyz="${x*(base_length/2-extrusion_length/2-extrusion_edge_to_base_edge)} ${y*base_width/2} ${base_height-extrusion_height/2}" rpy="0 0 0"/>
       <parent link="base_link"/>
       <child link="${prefix}_extrusion"/>

File: src/bigrdigr_description/urdf/sensors/camera.urdf.xacro (robot description, xacro)
@@ -5,6 +5,7 @@
 	<xacro:property name="pseye_camera_length" value="0.07" />
 	<xacro:property name="pseye_camera_width" value="0.09" />
+  <xacro:property name="pseye_camera_angle" value=".5236" /> <!--rad from horizontal, + = downward-->
   <xacro:property name="pseye_FOV" value="1.309"/> <!--56 or 75 degrees, need rad-->
-  <xacro:macro name="camera_link" params="number">
+  <xacro:macro name="camera_link" params="number extrusion">
     <link name="pseye_camera${number}">
       <visual>
@@ -23,8 +24,8 @@
     </link>
   </xacro:macro>
-  <xacro:macro name="camera_joint" params="number x y spin">
+  <xacro:macro name="camera_joint" params="number y spin extrusion">
     <joint name="camera${number}_joint" type="fixed">
-      <origin xyz="${x*(base_length/2-pseye_camera_length/2)} ${y*(base_width/2+pseye_camera_width/2)} ${base_height-pseye_camera_height/2}" rpy="0 0 ${spin}"/>
-      <parent link="base_link"/>
+      <origin xyz="0 ${y*(extrusion_width-pseye_camera_width/2)} ${0-extrusion_height/2-pseye_camera_height/2}" rpy="0 ${pseye_camera_angle} ${spin}"/>
+      <parent link="${extrusion}"/>
       <child link="pseye_camera${number}"/>
     </joint>
@@ -71,7 +72,7 @@
   	</gazebo>
   </xacro:macro>
-  <xacro:macro name="camera_macro" params="number x y spin">
-    <camera_link number="${number}"/>
-    <camera_joint number="${number}" x="${x}" y="${y}" spin="${spin}"/>
+  <xacro:macro name="camera_macro" params="number y extrusion spin">
+    <camera_link number="${number}" extrusion="${extrusion}"/>
+    <camera_joint number="${number}" y="${y}" spin="${spin}" extrusion="${extrusion}"/>
     <camera_gazebo number="${number}"/>
   </xacro:macro>

File: src/bigrdigr_description/urdf/sensors/imu.urdf.xacro (robot description, xacro)
@@ -6,10 +6,10 @@
   <xacro:property name="imu_height" value="0.01" />
   <xacro:property name="imu_visual" value="true"/>
-  <xacro:macro name="imu_joint" params="number">
+  <xacro:macro name="imu_joint" params="number x y extrusion">
     <joint name="imu${number}_joint" type="fixed">
       <axis rpy="0 0 0" xyz="0 1 0"/>
-      <parent link="base_link" />
+      <parent link="${extrusion}" />
       <child link="imu${number}_link" />
-      <origin xyz="0 0 ${base_height + imu_height/2.0}" rpy="0 0 0" />
+      <origin xyz="${x*(extrusion_length/2+imu_length/2)} ${y*extrusion_width/2} 0" rpy="0 0 0" />
     </joint>
   </xacro:macro>
@@ -53,6 +53,6 @@
   	</gazebo>
   </xacro:macro>
-  <xacro:macro name="imu" params="number">
-    <imu_joint number="${number}"/>
+  <xacro:macro name="imu" params="number x y extrusion">
+    <imu_joint number="${number}" x="${x}" y="${y}" extrusion="${extrusion}"/>
     <imu_link number="${number}"/>
     <imu_gazebo number="${number}"/>

File: src/bigrdigr_description/urdf/wheel.urdf.xacro (robot description, xacro)
@@ -57,8 +57,8 @@
       <type>transmission_interface/SimpleTransmission</type>
       <joint name="${prefix}_wheel_joint">
-        <hardwareInterface>hardware_interface/EffortJointInterface</hardwareInterface>
+        <hardwareInterface>hardware_interface/VelocityJointInterface</hardwareInterface>
       </joint>
       <actuator name="${prefix}_wheel_motor">
-        <hardwareInterface>EffortJointInterface</hardwareInterface>
+        <hardwareInterface>hardware_interface/VelocityJointInterface</hardwareInterface>
         <mechanicalReduction>1</mechanicalReduction>
       </actuator>

Commit message: bigrdigr_control formatter_string Made telecom direct work, no auton

File: src/bigrdigr_description/urdf/bigrdigr.urdf.xacro (robot description, xacro)
@@ -67,5 +67,5 @@
 	<!-- world_origin is a fictitious link(frame) that is on the ground right below base_link origin -->
 	<!-- z axis is height -->
-	<link name="world_origin"/>
+  <!--<link name="world_origin"/>
   <gazebo reference="world_origin">
 		<turnGravityOff>false</turnGravityOff>
@@ -75,5 +75,5 @@
 		<parent link="world_origin" />
 		<child link="base_link" />
-	</joint>
+  </joint> -->
 	<link name="base_link">
 		<visual>

File: src/bigrdigr_description/urdf/sensors/imu.urdf.xacro (robot description, xacro)
@@ -6,4 +6,5 @@
   <xacro:property name="imu_height" value="0.01" />
   <xacro:property name="imu_visual" value="true"/>
+  <xacro:property name="pi" value="3.1415"/>
   <xacro:macro name="imu_joint" params="number x y extrusion">
     <joint name="imu${number}_joint" type="fixed">
@@ -11,5 +12,5 @@
       <parent link="${extrusion}" />
       <child link="imu${number}_link" />
-      <origin xyz="${x*(extrusion_length/2+imu_length/2)} ${y*extrusion_width/2} 0" rpy="0 0 0" />
+      <origin xyz="${x*(extrusion_length/2+imu_length/2)} ${y*extrusion_width/2} 0" rpy="${pi} 0 0" />
     </joint>
   </xacro:macro>
