Commit message: Cleaned up some of the URDF descriptions and added clarifying comments

File: src/bigrdigr_description/urdf/bigrdigr.urdf.xacro (robot description, xacro)
@@ -26,5 +26,5 @@
     <color rgba="0.8 0.2 0 1"/>
   </material>
-  <!-- Hard coded dimenstions well approximating robot -->
+  <!-- Hard coded dimenstions approximating robot -->
   <!-- Robot modeled as:
        a large box (base_link), origin at bottom,
@@ -33,190 +33,235 @@
        a box that reps the drum,
        four extensions with cameras, imus, decawaves,
-       two rgbd cams front and back center -->
-  <!-- red axis = x axis green axis = y blue axis = z -->
-  <!-- Equation for inertial matrix of box/prisim -->
-  <xacro:macro name="box_inertial_matrix" params="m l w h">
-  	<inertia ixx="${(m*(w*w+h*h))/12.0}" ixy = "0.0" ixz = "0.0"
-     				 iyy="${(m*(l*l+h*h))/12.0}" iyz = "0.0"
-     				 izz="${(m*(l*l+w*w))/12.0}" />
-  </xacro:macro>
-  <!-- Equation for inertial matrix of cylinder (rotating around y axis) -->
-  <xacro:macro name="cylinder_inertia" params="m r h">
-  	<inertia ixx="${(m*(3*r*r+h*h))/12.0}" ixy = "0.0" ixz = "0.0"
-     				 iyy="${m*r*r/2.0}"			   iyz = "0.0"
-     				 izz="${(m*(3*r*r+h*h))/12.0}"  />
-  </xacro:macro>
-  <!-- Main dimensions: meters, kg, seconds, rads -->
-  <xacro:property name="base_height" value="0.54" /> <!--z-->
-	<xacro:property name="base_length" value="0.864925" /> <!--x-->
-	<xacro:property name="base_width" value="0.740" /> <!--y-->
-	<xacro:property name="base_mass" value="72.0" />
-  <xacro:property name="leg_height" value="0.127"/>
-  <xacro:property name="leg_length" value="0.739775"/>
-  <xacro:property name="leg_width" value="0.0508"/>
-  <xacro:property name="leg_mass" value="4"/>
-  <xacro:property name="leg_x_origin_to_axle" value="${leg_length/2-.10835}" />
-	<xacro:property name="leg_y_origin_to_axle" value="0.0254" />
-	<xacro:property name="leg_axle_height" value="0.10535" />
-  <xacro:property name="drum_height" value=".11809"/>
-  <xacro:property name="drum_length" value="${base_length+.01}"/>
-  <xacro:property name="drum_width" value=".34"/>
-  <xacro:property name="drum_mass" value="2"/>
-  <xacro:property name="drum_y_origin_to_base_origin" value="${base_width/2-drum_width/2}"/>
-  <!-- World Origin -->
-	<!-- world_origin is a fictitious link(frame) that is on the ground right below base_link origin -->
-	<!-- z axis is height -->
-  <!--<link name="world_origin"/>
-  <gazebo reference="world_origin">
-		<turnGravityOff>false</turnGravityOff>
+       two rgbd(realsense) cams front and back center -->
+  <!-- red axis = x, axis green axis = y, blue axis = z -->
+  <!-- The following macros and properties are used to define the links
+       and joints of the bot -->
+    <!-- Equation for inertial matrix of box/prisim -->
+    <xacro:macro name="box_inertial_matrix" params="m l w h">
+    	<inertia ixx="${(m*(w*w+h*h))/12.0}" ixy = "0.0" ixz = "0.0"
+       				 iyy="${(m*(l*l+h*h))/12.0}" iyz = "0.0"
+       				 izz="${(m*(l*l+w*w))/12.0}" />
+    </xacro:macro>
+    <!-- Equation for inertial matrix of cylinder (rotating around y axis) -->
+    <xacro:macro name="cylinder_inertia" params="m r h">
+    	<inertia ixx="${(m*(3*r*r+h*h))/12.0}" ixy = "0.0" ixz = "0.0"
+       				 iyy="${m*r*r/2.0}"			   iyz = "0.0"
+       				 izz="${(m*(3*r*r+h*h))/12.0}"  />
+    </xacro:macro>
+    <!-- Main dimensions: meters, kg, seconds, rads -->
+    <xacro:property name="base_height" value="0.54" /> <!--z-->
+	  <xacro:property name="base_length" value="0.864925" /> <!--x-->
+	  <xacro:property name="base_width" value="0.740" /> <!--y-->
+	  <xacro:property name="base_mass" value="72.0" />
+    <xacro:property name="leg_height" value="0.127"/>
+    <xacro:property name="leg_length" value="0.739775"/>
+    <xacro:property name="leg_width" value="0.0508"/>
+    <xacro:property name="leg_mass" value="4"/>
+    <xacro:property name="leg_x_origin_to_axle" value="${leg_length/2-.10835}" />
+	  <xacro:property name="leg_y_origin_to_axle" value="0.0254" />
+	  <xacro:property name="leg_axle_height" value="0.10535" />
+    <xacro:property name="drum_height" value=".11809"/>
+    <xacro:property name="drum_length" value="${base_length+.01}"/>
+    <xacro:property name="drum_width" value=".34"/>
+    <xacro:property name="drum_mass" value="2"/>
+    <xacro:property name="drum_y_origin_to_base_origin" value="${base_width/2-drum_width/2}"/>
+  <!-- End macros and properties -->
+  <!-- The following links and joints define the robots components
+       and their relationship to eachother -->
+    <!-- BASE_LINK represent the frame of the robot -->
+	    <link name="base_link">
+		    <!-- visual is the model shown in gazebo / rviz -->
+		    <visual>
+			    <origin xyz="0 0 ${base_height/2.0}" rpy="0 0 0"/>
+			    <geometry>
+				    <box size=" ${base_length} ${base_width} ${base_height}" />
+			    </geometry>
+			    <material name="grey"/>
+		    </visual>
+        <!-- collision and inertial are used by the physics model used
+             in simulation -->
+		    <collision>
+			    <origin xyz="0 0 ${base_height/2.0}" rpy="0 0 0"/>
+			    <geometry>
+				    <box size="${base_length} ${base_width} ${base_width}"/>
+			    </geometry>
+		    </collision>
+		    <inertial>
+			    <origin xyz="0 0 ${base_height/2.0}" rpy="0 0 0"/>
+			    <mass value="${base_mass}"/>
+			    <box_inertial_matrix m="${base_mass}" h="${base_height}" l="${base_length}" w="${base_width}" />
+		    </inertial>
+	    </link>
+      <!-- Gazebo element covers assigning values not handled by the URDF file format -->
+      <gazebo reference="base_link">
+        <material>Gazebo/Grey</material>
+        <turnGravityOff>false</turnGravityOff>
+      </gazebo>
+    <!-- End base_link(robot frame) description -->
+    <!-- Attaching the left drivetrain to the robot frame -->
+      <!-- joint defines position relationship of the child to the parent-->
+      <joint name="left_leg_joint" type="fixed">
+		    <origin xyz="0 ${base_width/2-leg_width/2} ${-leg_height}" rpy="0 0 0" />
+		    <parent link="base_link" />
+		    <child link="left_leg" />
+	    </joint>
+      <!-- LEFT_LEG represents the left of the drive train -->
+	    <link name="left_leg">
+		    <!-- visual is the model shown in gazebo / rviz -->
+		    <visual>
+			    <origin xyz="0 0 ${leg_height/2.0}" rpy="0 0 0"/>
+			    <geometry>
+				    <box size=" ${leg_length} ${leg_width} ${leg_height}" />
+			    </geometry>
+			    <material name="blue"/>
+		    </visual>
+        <!-- collision and inertial are used by the physics model used
+             in simulation -->
+		    <collision>
+			    <origin xyz="0 0 ${leg_height/2.0}" rpy="0 0 0"/>
+			    <geometry>
+				    <box size="${leg_length} ${leg_width} ${leg_width}"/>
+			    </geometry>
+		    </collision>
+		    <inertial>
+			    <origin xyz="0 0 ${leg_height/2.0}" rpy="0 0 0"/>
+			    <mass value="${leg_mass}"/>
+			    <box_inertial_matrix m="${leg_mass}" h="${leg_height}" l="${leg_length}" w="${leg_width}" />
+		    </inertial>
+	    </link>
+      <!-- Gazebo element covers assigning values not handled by the URDF file format -->
+      <gazebo reference="left_leg">
+        <material>Gazebo/Blue</material>
+        <turnGravityOff>false</turnGravityOff>
+      </gazebo>
+    <!-- End left_leg_joint(left drive train) description -->
+    <!-- Attaching the right drivetrain to the robot frame -->
+      <!-- joint defines position relationship of the child to the parent-->
+      <joint name="right_leg_joint" type="fixed">
+        <origin xyz="0 ${-base_width/2+leg_width/2} ${-leg_height}" rpy="0 0 0" />
+        <parent link="base_link" />
+        <child link="right_leg" />
+      </joint>
+      <!-- RIGHT_LEG represents the left of the drive train -->
+      <link name="right_leg">
+        <!-- visual is the model shown in gazebo / rviz -->
+        <visual>
+          <origin xyz="0 0 ${leg_height/2.0}" rpy="0 0 0"/>
+          <geometry>
+            <box size=" ${leg_length} ${leg_width} ${leg_height}" />
+          </geometry>
+          <material name="blue"/>
+        </visual>
+        <!-- collision and inertial are used by the physics model used
+             in simulation -->
+        <collision>
+          <origin xyz="0 0 ${leg_height/2.0}" rpy="0 0 0"/>
+          <geometry>
+            <box size="${leg_length} ${leg_width} ${leg_width}"/>
+          </geometry>
+        </collision>
+        <inertial>
+          <origin xyz="0 0 ${leg_height/2.0}" rpy="0 0 0"/>
+          <mass value="${leg_mass}"/>
+          <box_inertial_matrix m="${leg_mass}" h="${leg_height}" l="${leg_length}" w="${leg_width}" />
+        </inertial>
+      </link>
+      <!-- Gazebo element covers assigning values not handled by the URDF file format -->
+      <gazebo reference="right_leg">
+        <material>Gazebo/Blue</material>
+        <turnGravityOff>false</turnGravityOff>
+      </gazebo>
+    <!-- End right_leg_joint(right drive train) description -->
+    <!-- Attaching the drum to the robot frame -->
+    <!-- joint defines position relationship of the child to the parent-->
+    <joint name="drum_joint" type="fixed">
+		  <origin xyz="0 ${drum_y_origin_to_base_origin} ${-drum_height/2}" rpy="0 0 0" />
+		  <parent link="base_link" />
+		  <child link="drum" />
+	  </joint>
+    <!-- DRUM represents the digging wheel -->
+	  <link name="drum">
+      <!-- visual is the model shown in gazebo / rviz -->
+      <visual>
+        <origin xyz="0 0 0" rpy="0 0 0"/>
+        <geometry>
+          <box size=" ${drum_length} ${drum_width} ${drum_height}" />
+        </geometry>
+        <material name="purple"/>
+      </visual>
+      <!-- collision and inertial are used by the physics model used
+           in simulation -->
+      <collision>
+        <origin xyz="0 0 0" rpy="0 0 0"/>
+        <geometry>
+          <box size="${drum_length} ${drum_width} ${drum_width}"/>
+        </geometry>
+      </collision>
+      <inertial>
+        <origin xyz="0 0 0" rpy="0 0 0"/>
+        <mass value="${drum_mass}"/>
+        <box_inertial_matrix m="${drum_mass}" h="${drum_height}" l="${drum_length}" w="${drum_width}" />
+      </inertial>
+	  </link>
+    <!-- Gazebo element covers assigning values not handled by the URDF file format -->
+    <gazebo reference="drum">
+      <material>Gazebo/Purple</material>
+      <turnGravityOff>false</turnGravityOff>
+    </gazebo>
+    <!-- End drum description -->
+  <!-- End links and joints -->
+  <!-- The following represent extrusions from the frame and drivetrain
+       which are defined in wheel.urdf.xacro and extrusion.urdf.xacro -->
+    <!-- wheels -->
+    <wheel prefix="front_left" leg="left_leg" x="1" y="1"/>
+    <wheel prefix="front_right" leg="right_leg" x="1" y="-1"/>
+    <wheel prefix="back_left" leg="left_leg" x="-1" y="1"/>
+    <wheel prefix="back_right" leg="right_leg" x="-1" y="-1"/>
+    <!-- extrusions for cameras / sensors -->
+    <extrusion prefix="front_left" x="1" y="1"/>
+    <extrusion prefix="front_right" x="1" y="-1"/>
+    <extrusion prefix="back_left" x="-1" y="1"/>
+    <extrusion prefix="back_right" x="-1" y="-1"/>
+  <!-- End wheels and extrusions -->
+  <!-- The following represent the camera placementon the extrusions -->
+    <xacro:arg name="cameras" default="false"/>
+    <xacro:property name="useCams" value="$(arg cameras)"/>
+    <xacro:if value="${useCams == 'true'}">
+      <camera_macro number="1" y="1" extrusion="front_left_extrusion" spin="0"/>
+      <camera_macro number="2" y="-1" extrusion="front_right_extrusion" spin="0"/>
+      <camera_macro number="3" y="1" extrusion="back_left_extrusion" spin="${PI}"/>
+      <camera_macro number="4" y="-1" extrusion="back_right_extrusion" spin="${PI}"/>
+    </xacro:if>
+  <!-- End cameras -->
+  <!-- The following defines the positions of the IMU and Decawave sensors -->
+    <!-- imu and deca front left, back right. in front of extrusion -->
+    <imu number="1" x="1" y="1" extrusion="front_left_extrusion"/>
+    <imu number="2" x="1" y="-1" extrusion="back_right_extrusion"/>
+  <!-- End sensors -->
+  <!-- skid steer plugin handles driving for us -->
+	<gazebo>
+	  <plugin name="skid_steer_drive_controller" filename="libgazebo_ros_skid_steer_drive.so">
+	    <updateRate>100.0</updateRate>
+	    <robotNamespace>/bigrdigr</robotNamespace>
+			<commandTopic>cmd_vel</commandTopic>
+			<odometryTopic>odometry/wheel</odometryTopic>
+	    <leftFrontJoint>front_left_wheel_joint</leftFrontJoint>
+	    <rightFrontJoint>front_right_wheel_joint</rightFrontJoint>
+	    <leftRearJoint>back_left_wheel_joint</leftRearJoint>
+	    <rightRearJoint>back_right_wheel_joint</rightRearJoint>
+	    <wheelSeparation>${2*base_width}</wheelSeparation>
+	    <wheelDiameter>${2*wheel_radius}</wheelDiameter>
+	    <robotBaseFrame>base_link</robotBaseFrame>
+	    <torque>20</torque>
+	    <broadcastTF>true</broadcastTF>
+			<legacyMode>false</legacyMode>
+	  </plugin>
 	</gazebo>
-	<joint name="base_footprint_joint" type="fixed">
-		<origin xyz="0 0 ${leg_height-leg_axle_height}" rpy="0 0 0" />
-		<parent link="world_origin" />
-		<child link="base_link" />
-  </joint> -->
-	<link name="base_link">
-		<visual>
-			<origin xyz="0 0 ${base_height/2.0}" rpy="0 0 0"/>
-			<geometry>
-				<box size=" ${base_length} ${base_width} ${base_height}" />
-			</geometry>
-			<material name="grey"/>
-		</visual>
-		<collision>
-			<origin xyz="0 0 ${base_height/2.0}" rpy="0 0 0"/>
-			<geometry>
-				<box size="${base_length} ${base_width} ${base_width}"/>
-			</geometry>
-		</collision>
-		<inertial>
-			<origin xyz="0 0 ${base_height/2.0}" rpy="0 0 0"/>
-			<mass value="${base_mass}"/>
-			<box_inertial_matrix m="${base_mass}" h="${base_height}" l="${base_length}" w="${base_width}" />
-		</inertial>
-	</link>
-  <gazebo reference="base_link">
-    <material>Gazebo/Grey</material>
-    <turnGravityOff>false</turnGravityOff>
-  </gazebo>
-  <joint name="left_leg_joint" type="fixed">
-		<origin xyz="0 ${base_width/2-leg_width/2} ${-leg_height}" rpy="0 0 0" />
-		<parent link="base_link" />
-		<child link="left_leg" />
-	</joint>
-	<link name="left_leg">
-		<visual>
-			<origin xyz="0 0 ${leg_height/2.0}" rpy="0 0 0"/>
-			<geometry>
-				<box size=" ${leg_length} ${leg_width} ${leg_height}" />
-			</geometry>
-			<material name="blue"/>
-		</visual>
-		<collision>
-			<origin xyz="0 0 ${leg_height/2.0}" rpy="0 0 0"/>
-			<geometry>
-				<box size="${leg_length} ${leg_width} ${leg_width}"/>
-			</geometry>
-		</collision>
-		<inertial>
-			<origin xyz="0 0 ${leg_height/2.0}" rpy="0 0 0"/>
-			<mass value="${leg_mass}"/>
-			<box_inertial_matrix m="${leg_mass}" h="${leg_height}" l="${leg_length}" w="${leg_width}" />
-		</inertial>
-	</link>
-  <gazebo reference="left_leg">
-    <material>Gazebo/Blue</material>
-    <turnGravityOff>false</turnGravityOff>
-  </gazebo>
-  <joint name="right_leg_joint" type="fixed">
-    <origin xyz="0 ${-base_width/2+leg_width/2} ${-leg_height}" rpy="0 0 0" />
-    <parent link="base_link" />
-    <child link="right_leg" />
-  </joint>
-  <link name="right_leg">
-    <visual>
-      <origin xyz="0 0 ${leg_height/2.0}" rpy="0 0 0"/>
-      <geometry>
-        <box size=" ${leg_length} ${leg_width} ${leg_height}" />
-      </geometry>
-      <material name="blue"/>
-    </visual>
-    <collision>
-      <origin xyz="0 0 ${leg_height/2.0}" rpy="0 0 0"/>
-      <geometry>
-        <box size="${leg_length} ${leg_width} ${leg_width}"/>
-      </geometry>
-    </collision>
-    <inertial>
-      <origin xyz="0 0 ${leg_height/2.0}" rpy="0 0 0"/>
-      <mass value="${leg_mass}"/>
-      <box_inertial_matrix m="${leg_mass}" h="${leg_height}" l="${leg_length}" w="${leg_width}" />
-    </inertial>
-  </link>
-  <gazebo reference="right_leg">
-    <material>Gazebo/Blue</material>
-    <turnGravityOff>false</turnGravityOff>
-  </gazebo>
-  <wheel prefix="front_left" leg="left_leg" x="1" y="1"/>
-  <wheel prefix="front_right" leg="right_leg" x="1" y="-1"/>
-  <wheel prefix="back_left" leg="left_leg" x="-1" y="1"/>
-  <wheel prefix="back_right" leg="right_leg" x="-1" y="-1"/>
-  <extrusion prefix="front_left" x="1" y="1"/>
-  <extrusion prefix="front_right" x="1" y="-1"/>
-  <extrusion prefix="back_left" x="-1" y="1"/>
-  <extrusion prefix="back_right" x="-1" y="-1"/>
-  <!-- cameras under extrusions -->
-  <xacro:arg name="cameras" default="false"/>
-  <xacro:property name="useCams" value="$(arg cameras)"/>
-  <xacro:if value="${useCams == 'true'}">
-    <camera_macro number="1" y="1" extrusion="front_left_extrusion" spin="0"/>
-    <camera_macro number="2" y="-1" extrusion="front_right_extrusion" spin="0"/>
-    <camera_macro number="3" y="1" extrusion="back_left_extrusion" spin="${PI}"/>
-    <camera_macro number="4" y="-1" extrusion="back_right_extrusion" spin="${PI}"/>
-  </xacro:if>
-  <!-- imu and deca front left, back right. in front of extrusion -->
-  <imu number="1" x="1" y="1" extrusion="front_left_extrusion"/>
-  <imu number="2" x="1" y="-1" extrusion="back_right_extrusion"/>
-  <joint name="drum_joint" type="prismatic">
-		<origin xyz="0 ${drum_y_origin_to_base_origin} ${-drum_height/2}" rpy="0 0 0" />
-		<parent link="base_link" />
-		<child link="drum" />
-    <axis xyz="0 0 1"/>
-    <dynamics damping="0.1" friction="0.1"/> <!-- get real Ns/m damping N friction -->
-    <limit lower="0" upper="${base_height}" effort="1000" velocity="10"/> <!-- m distance, max effort and vel -->
-	</joint>
-	<link name="drum">
-    <visual>
-      <origin xyz="0 0 0" rpy="0 0 0"/>
-      <geometry>
-        <box size=" ${drum_length} ${drum_width} ${drum_height}" />
-      </geometry>
-      <material name="purple"/>
-    </visual>
-    <collision>
-      <origin xyz="0 0 0" rpy="0 0 0"/>
-      <geometry>
-        <box size="${drum_length} ${drum_width} ${drum_width}"/>
-      </geometry>
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
File: src/bigrdigr_description/urdf/extrusion.urdf.xacro (robot description, xacro)
@@ -1,45 +1,56 @@
 <?xml version="1.0" encoding="UTF-8"?>
 <robot name="bigrdigr" xmlns:xacro="https://www.ros.org/wiki/xacro">
-  <!-- Main dimensions: meters, kg, seconds, rads -->
-  <xacro:property name="extrusion_height" value="0.0254"/>
-  <xacro:property name="extrusion_length" value="0.0254"/>
-  <xacro:property name="extrusion_width" value="0.13254"/>
-  <xacro:property name="extrusion_mass" value="0.5"/>
-  <xacro:property name="extrusion_edge_to_base_edge" value="0.0946"/>
-  <xacro:macro name="extrusion_joint" params="prefix x y">
-    <joint name="${prefix}_extrusion_joint" type="fixed">
-      <origin xyz="${x*(base_length/2-extrusion_length/2-extrusion_edge_to_base_edge)} ${y*base_width/2} ${base_height-extrusion_height/2}" rpy="0 0 0"/>
-      <parent link="base_link"/>
-      <child link="${prefix}_extrusion"/>
-  	</joint>
-  </xacro:macro>
-  <xacro:macro name="extrusion_link" params="prefix y">
-  	<link name="${prefix}_extrusion">
-  		<visual>
-  			<origin xyz="0 ${y*extrusion_width/2} 0" rpy="0 0 0"/>
-  			<geometry>
-  				<box size=" ${extrusion_length} ${extrusion_width} ${extrusion_height}" />
-  			</geometry>
-  			<material name="green"/>
-  		</visual>
-  		<collision>
-  			<origin xyz="0 ${y*extrusion_width/2} 0" rpy="0 0 0"/>
-  			<geometry>
-          <box size=" ${extrusion_length} ${extrusion_width} ${extrusion_height}" />
-  			</geometry>
-  		</collision>
-  		<inertial>
-  			<origin xyz="0 0 ${leg_height/2.0}" rpy="0 0 0"/>
-  			<mass value="${leg_mass}"/>
-  			<box_inertial_matrix m="${leg_mass}" h="${leg_height}" l="${leg_length}" w="${leg_width}" />
-  		</inertial>
-  	</link>
-  </xacro:macro>
-  <xacro:macro name="extrusion_gazebo" params="prefix">
-    <gazebo reference="${prefix}_extrusion">
-      <material>Gazebo/Green</material>
-      <turnGravityOff>false</turnGravityOff>
-    </gazebo>
-  </xacro:macro>
+  <!-- Properties describe size of sensor boxes located at corners of
+       the robot's frame -->
+    <!-- Main dimensions: meters, kg, seconds, rads -->
+    <xacro:property name="extrusion_height" value="0.0254"/>
+    <xacro:property name="extrusion_length" value="0.0254"/>
+    <xacro:property name="extrusion_width" value="0.13254"/>
+    <xacro:property name="extrusion_mass" value="0.5"/>
+    <xacro:property name="extrusion_edge_to_base_edge" value="0.0946"/>
+  <!-- End properties -->
+  <!-- Attaching extrusions(sensor boxes) to the frame -->
+    <!-- Macro which creates joints for the sensor boxes -->
+    <xacro:macro name="extrusion_joint" params="prefix x y">
+      <joint name="${prefix}_extrusion_joint" type="fixed">
+        <origin xyz="${x*(base_length/2-extrusion_length/2-extrusion_edge_to_base_edge)} ${y*base_width/2} ${base_height-extrusion_height/2}" rpy="0 0 0"/>
+        <parent link="base_link"/>
+        <child link="${prefix}_extrusion"/>
+    	</joint>
+    </xacro:macro>
+    <!-- Macro which creates links for the sensor boxes -->
+    <xacro:macro name="extrusion_link" params="prefix y">
+    	<link name="${prefix}_extrusion">
+    		<!-- visual is the model shown in gazebo / rviz -->
+    		<visual>
+    			<origin xyz="0 ${y*extrusion_width/2} 0" rpy="0 0 0"/>
+    			<geometry>
+    				<box size=" ${extrusion_length} ${extrusion_width} ${extrusion_height}" />
+    			</geometry>
+    			<material name="green"/>
+    		</visual>
+        <!-- collision and inertial are used by the physics model used
+             in simulation -->
+    		<collision>
+    			<origin xyz="0 ${y*extrusion_width/2} 0" rpy="0 0 0"/>
+    			<geometry>
+            <box size=" ${extrusion_length} ${extrusion_width} ${extrusion_height}" />
+    			</geometry>
+    		</collision>
+    		<inertial>
+    			<origin xyz="0 0 ${leg_height/2.0}" rpy="0 0 0"/>
+    			<mass value="${leg_mass}"/>
+    			<box_inertial_matrix m="${leg_mass}" h="${leg_height}" l="${leg_length}" w="${leg_width}" />
+    		</inertial>
+    	</link>
+    </xacro:macro>
+    <xacro:macro name="extrusion_gazebo" params="prefix">
+      <gazebo reference="${prefix}_extrusion">
+        <material>Gazebo/Green</material>
+        <turnGravityOff>false</turnGravityOff>
+      </gazebo>
+    </xacro:macro>
+  <!-- End extrusion description -->
+  <!-- Generic extrusion creation, possibly not needed? -->
   <xacro:macro name="extrusion" params="prefix x y">
     <extrusion_link prefix="${prefix}" y="${y}"/>
