Commit message: change dimensions of rovr

File: src/rovr_description/urdf/rovr.urdf.xacro (robot description, xacro)
@@ -50,18 +50,22 @@
     </xacro:macro>
     <!-- Main dimensions: meters, kg, seconds, rads -->
-    <xacro:property name="base_height" value="0.54" /> <!--z-->
-	  <xacro:property name="base_length" value="0.864925" /> <!--x-->
-	  <xacro:property name="base_width" value="0.740" /> <!--y-->
+    <!-- Rectangular Body Frame-->
+    <xacro:property name="base_height" value=".500" /> <!--z-->
+	  <xacro:property name="base_length" value="0.500" /> <!--x-->
+	  <xacro:property name="base_width" value="0.7808" /> <!--y-->
 	  <xacro:property name="base_mass" value="72.0" />
-    <xacro:property name="leg_height" value="0.127"/>
+    <!--Part that extends from Body (Blue)-->
+    <xacro:property name="leg_height" value=".0635"/>
     <xacro:property name="leg_length" value="0.739775"/>
     <xacro:property name="leg_width" value="0.0508"/>
     <xacro:property name="leg_mass" value="4"/>
+    <!--Distance from Leg to Center-->
     <xacro:property name="leg_x_origin_to_axle" value="${leg_length/2-.10835}" />
 	  <xacro:property name="leg_y_origin_to_axle" value="0.0254" />
 	  <xacro:property name="leg_axle_height" value="0.10535" />
-    <xacro:property name="drum_height" value=".11809"/>
+    <!-- Rectangular representation of Drum (Purple)-->
+    <xacro:property name="drum_height" value=".0635"/>
     <xacro:property name="drum_length" value="${base_length+.01}"/>
-    <xacro:property name="drum_width" value=".34"/>
+    <xacro:property name="drum_width" value=".110"/>
     <xacro:property name="drum_mass" value="2"/>
     <xacro:property name="drum_y_origin_to_base_origin" value="${base_width/2-drum_width/2}"/>
@@ -219,10 +223,13 @@
     <wheel prefix="back_right" leg="right_leg" x="-1" y="-1"/>
     <!-- extrusions for cameras / sensors -->
+    <!--
     <extrusion prefix="front_left" x="1" y="1"/>
     <extrusion prefix="front_right" x="1" y="-1"/>
     <extrusion prefix="back_left" x="-1" y="1"/>
     <extrusion prefix="back_right" x="-1" y="-1"/>
+    -->
   <!-- End wheels and extrusions -->
   <!-- The following represent the camera placementon the extrusions -->
+  <!--
     <xacro:arg name="cameras" default="false"/>
     <xacro:property name="useCams" value="$(arg cameras)"/>
@@ -233,4 +240,5 @@
       <camera_macro number="4" y="-1" extrusion="back_right_extrusion" spin="${PI}"/>
     </xacro:if>
+    -->
   <!-- End cameras -->
   <!-- The following defines the positions of the IMU and Decawave sensors -->

File: src/rovr_description/urdf/wheel.urdf.xacro (robot description, xacro)
@@ -4,6 +4,6 @@
 	  <!-- Main dimensions: meters, kg, seconds, rads -->
 	  <xacro:property name="PI" value="3.141592653589793238462643383279502884197" />
-	  <xacro:property name="wheel_width" value=".15" />
-	  <xacro:property name="wheel_radius" value=".18035" />
+	  <xacro:property name="wheel_width" value=".1" />
+	  <xacro:property name="wheel_radius" value=".245" />
 	  <xacro:property name="wheel_mass" value="2" />
   <!-- end properties -->

Commit message: change dimensions of rovr

File: src/rovr_description/urdf/rovr.urdf.xacro (robot description, xacro)
@@ -52,22 +52,24 @@
     </xacro:macro>
     <!-- Main dimensions: meters, kg, seconds, rads -->
-    <xacro:property name="base_height" value="0.54" /> <!--z-->
-	  <xacro:property name="base_length" value="0.740" /> <!--x--> <!-- 0.864925 -->
-	  <xacro:property name="base_width" value="0.864925" /> <!--y--> <!-- 0.740 -->
+    <!-- Rectangular Body Frame-->
+    <xacro:property name="base_height" value=".500" /> <!--z-->
+	  <xacro:property name="base_length" value="0.500" /> <!--x-->
+	  <xacro:property name="base_width" value="0.7808" /> <!--y-->
 	  <xacro:property name="base_mass" value="72.0" />
-    <xacro:property name="leg_height" value="0.127"/>
+    <!--Part that extends from Body (Blue)-->
+    <xacro:property name="leg_height" value=".0635"/>
     <xacro:property name="leg_length" value="0.739775"/>
     <xacro:property name="leg_width" value="0.0508"/>
     <xacro:property name="leg_mass" value="4"/>
-    <xacro:property name="leg_x_origin_to_axle" value="${leg_length/2-.1778}" />
+    <!--Distance from Leg to Center-->
+    <xacro:property name="leg_x_origin_to_axle" value="${leg_length/2-.10835}" />
 	  <xacro:property name="leg_y_origin_to_axle" value="0.0254" />
 	  <xacro:property name="leg_axle_height" value="0.10535" />
-    <xacro:property name="drum_height" value=".11809"/>
+    <!-- Rectangular representation of Drum (Purple)-->
+    <xacro:property name="drum_height" value=".0635"/>
     <xacro:property name="drum_length" value="${base_length+.01}"/>
-    <xacro:property name="drum_width" value=".34"/>
+    <xacro:property name="drum_width" value=".110"/>
     <xacro:property name="drum_mass" value="2"/>
     <xacro:property name="drum_y_origin_to_base_origin" value="${base_width/2-drum_width/2}"/>
-    <xacro:property name="realsense_front_offset" value="-0.0016"/>
-    <xacro:property name="realsense_back_offset" value="0.0429"/>
   <!-- End macros and properties -->
   <!-- The following links and joints define the robots components
@@ -223,10 +225,13 @@
     <wheel prefix="back_right" leg="right_leg" x="-1" y="-1"/>
     <!-- extrusions for cameras / sensors -->
+    <!--
     <extrusion prefix="front_left" x="1" y="1"/>
     <extrusion prefix="front_right" x="1" y="-1"/>
     <extrusion prefix="back_left" x="-1" y="1"/>
     <extrusion prefix="back_right" x="-1" y="-1"/>
+    -->
   <!-- End wheels and extrusions -->
-  <!-- The following represent the camera placement on the extrusions -->
+  <!-- The following represent the camera placementon the extrusions -->
+  <!--
     <xacro:arg name="cameras" default="false"/>
     <xacro:property name="useCams" value="$(arg cameras)"/>
@@ -237,4 +242,5 @@
       <camera_macro number="4" y="-1" extrusion="back_right_extrusion" spin="${PI}"/>
     </xacro:if>
+    -->
   <!-- End cameras -->
   <!-- The following defines the realsense placement on the frame -->

Commit message: direction reorientation

File: src/rovr_description/urdf/rovr.urdf.xacro (robot description, xacro)
@@ -42,5 +42,5 @@
     <xacro:macro name="box_inertial_matrix" params="m l w h">
     	<inertia ixx="${(m*(w*w+h*h))/12.0}" ixy = "0.0" ixz = "0.0"
-       				 iyy="${(m*(l*l+h*h))/12.0}" iyz = "0.0"
+       				 iyy="${(m*(l*l+h*h))/12.0}" iyz = "-1*base_width/20.0"
        				 izz="${(m*(l*l+w*w))/12.0}" />
     </xacro:macro>
@@ -52,12 +52,12 @@
     </xacro:macro>
     <!-- Main dimensions: meters, kg, seconds, rads -->
-    <!-- Rectangular Body Frame-->
-    <xacro:property name="base_height" value=".500" /> <!--z-->
-	  <xacro:property name="base_length" value="0.500" /> <!--x-->
+    <!-- Rectangular Body Frame (Gray)-->
+    <xacro:property name="base_height" value="0.500" /> <!--z-->
+	  <xacro:property name="base_length" value=".500" /> <!--x-->
 	  <xacro:property name="base_width" value="0.7808" /> <!--y-->
 	  <xacro:property name="base_mass" value="72.0" />
     <!--Part that extends from Body (Blue)-->
-    <xacro:property name="leg_height" value=".0635"/>
-    <xacro:property name="leg_length" value="0.739775"/>
+    <xacro:property name="leg_height" value="0.0635"/>
+    <xacro:property name="leg_length" value="${base_length}"/>
     <xacro:property name="leg_width" value="0.0508"/>
     <xacro:property name="leg_mass" value="4"/>
@@ -66,10 +66,11 @@
 	  <xacro:property name="leg_y_origin_to_axle" value="0.0254" />
 	  <xacro:property name="leg_axle_height" value="0.10535" />
-    <!-- Rectangular representation of Drum (Purple)-->
-    <xacro:property name="drum_height" value=".0635"/>
-    <xacro:property name="drum_length" value="${base_length+.01}"/>
-    <xacro:property name="drum_width" value=".110"/>
+    <!--Rectangular representation of Drum (Purple)-->
+    <xacro:property name="drum_height" value="0.0635"/>
+    <xacro:property name="drum_length" value="0.110"/>
+    <xacro:property name="drum_width" value="${base_width-2*leg_width}"/>
     <xacro:property name="drum_mass" value="2"/>
-    <xacro:property name="drum_y_origin_to_base_origin" value="${base_width/2-drum_width/2}"/>
+    <xacro:property name="drum_x_origin_to_base_origin" value=".195"/>
+    <xacro:property name="drum_y_origin_to_base_origin" value="0"s/>
   <!-- End macros and properties -->
   <!-- The following links and joints define the robots components
@@ -182,5 +183,5 @@
     <!-- joint defines position relationship of the child to the parent-->
     <joint name="drum_joint" type="fixed">
-		  <origin xyz="0 ${drum_y_origin_to_base_origin} ${-drum_height/2}" rpy="0 0 0" />
+		  <origin xyz="${drum_x_origin_to_base_origin} ${drum_y_origin_to_base_origin} ${-drum_height/2}" rpy="0 0 0" />
 		  <parent link="base_link" />
 		  <child link="drum" />
@@ -230,5 +231,6 @@
     <extrusion prefix="back_right" x="-1" y="-1"/>
   <!-- End wheels and extrusions -->
-  <!-- The following represent the camera placementon the extrusions -->
+  <!-- The following represent the camera placement on the extrusions -->
+  <!--
     <xacro:arg name="cameras" default="false"/>
     <xacro:property name="useCams" value="$(arg cameras)"/>

Commit message: direction reorientation

File: src/rovr_description/urdf/rovr.urdf.xacro (robot description, xacro)
@@ -40,5 +40,5 @@
     <xacro:macro name="box_inertial_matrix" params="m l w h">
     	<inertia ixx="${(m*(w*w+h*h))/12.0}" ixy = "0.0" ixz = "0.0"
-       				 iyy="${(m*(l*l+h*h))/12.0}" iyz = "0.0"
+       				 iyy="${(m*(l*l+h*h))/12.0}" iyz = "-1*base_width/20.0"
        				 izz="${(m*(l*l+w*w))/12.0}" />
     </xacro:macro>
@@ -50,12 +50,12 @@
     </xacro:macro>
     <!-- Main dimensions: meters, kg, seconds, rads -->
-    <!-- Rectangular Body Frame-->
-    <xacro:property name="base_height" value=".500" /> <!--z-->
-	  <xacro:property name="base_length" value="0.500" /> <!--x-->
+    <!-- Rectangular Body Frame (Gray)-->
+    <xacro:property name="base_height" value="0.500" /> <!--z-->
+	  <xacro:property name="base_length" value=".500" /> <!--x-->
 	  <xacro:property name="base_width" value="0.7808" /> <!--y-->
 	  <xacro:property name="base_mass" value="72.0" />
     <!--Part that extends from Body (Blue)-->
-    <xacro:property name="leg_height" value=".0635"/>
-    <xacro:property name="leg_length" value="0.739775"/>
+    <xacro:property name="leg_height" value="0.0635"/>
+    <xacro:property name="leg_length" value="${base_length}"/>
     <xacro:property name="leg_width" value="0.0508"/>
     <xacro:property name="leg_mass" value="4"/>
@@ -64,10 +64,11 @@
 	  <xacro:property name="leg_y_origin_to_axle" value="0.0254" />
 	  <xacro:property name="leg_axle_height" value="0.10535" />
-    <!-- Rectangular representation of Drum (Purple)-->
-    <xacro:property name="drum_height" value=".0635"/>
-    <xacro:property name="drum_length" value="${base_length+.01}"/>
-    <xacro:property name="drum_width" value=".110"/>
+    <!--Rectangular representation of Drum (Purple)-->
+    <xacro:property name="drum_height" value="0.0635"/>
+    <xacro:property name="drum_length" value="0.110"/>
+    <xacro:property name="drum_width" value="${base_width-2*leg_width}"/>
     <xacro:property name="drum_mass" value="2"/>
-    <xacro:property name="drum_y_origin_to_base_origin" value="${base_width/2-drum_width/2}"/>
+    <xacro:property name="drum_x_origin_to_base_origin" value=".195"/>
+    <xacro:property name="drum_y_origin_to_base_origin" value="0"s/>
   <!-- End macros and properties -->
   <!-- The following links and joints define the robots components
@@ -180,5 +181,5 @@
     <!-- joint defines position relationship of the child to the parent-->
     <joint name="drum_joint" type="fixed">
-		  <origin xyz="0 ${drum_y_origin_to_base_origin} ${-drum_height/2}" rpy="0 0 0" />
+		  <origin xyz="${drum_x_origin_to_base_origin} ${drum_y_origin_to_base_origin} ${-drum_height/2}" rpy="0 0 0" />
 		  <parent link="base_link" />
 		  <child link="drum" />
@@ -223,12 +224,10 @@
     <wheel prefix="back_right" leg="right_leg" x="-1" y="-1"/>
     <!-- extrusions for cameras / sensors -->
-    <!--
     <extrusion prefix="front_left" x="1" y="1"/>
     <extrusion prefix="front_right" x="1" y="-1"/>
     <extrusion prefix="back_left" x="-1" y="1"/>
     <extrusion prefix="back_right" x="-1" y="-1"/>
-    -->
   <!-- End wheels and extrusions -->
-  <!-- The following represent the camera placementon the extrusions -->
+  <!-- The following represent the camera placement on the extrusions -->
   <!--
     <xacro:arg name="cameras" default="false"/>

Commit message: Fix model wheel size

File: src/rovr_description/urdf/rovr.urdf.xacro (robot description, xacro)
@@ -56,6 +56,6 @@
 	  <xacro:property name="base_mass" value="72.0" />
     <!--Part that extends from Body (Blue)-->
-    <xacro:property name="leg_height" value=".0635"/>
-    <xacro:property name="leg_length" value="0.739775"/>
+    <xacro:property name="leg_height" value=".1"/>
+    <xacro:property name="leg_length" value="0.5"/>
     <xacro:property name="leg_width" value="0.0508"/>
     <xacro:property name="leg_mass" value="4"/>
@@ -65,5 +65,5 @@
 	  <xacro:property name="leg_axle_height" value="0.10535" />
     <!-- Rectangular representation of Drum (Purple)-->
-    <xacro:property name="drum_height" value=".0635"/>
+    <xacro:property name="drum_height" value=".0300"/>
     <xacro:property name="drum_length" value="${base_length+.01}"/>
     <xacro:property name="drum_width" value=".110"/>

File: src/rovr_description/urdf/wheel.urdf.xacro (robot description, xacro)
@@ -5,5 +5,5 @@
 	  <xacro:property name="PI" value="3.141592653589793238462643383279502884197" />
 	  <xacro:property name="wheel_width" value=".1" />
-	  <xacro:property name="wheel_radius" value=".245" />
+	  <xacro:property name="wheel_radius" value="0.1225" />
 	  <xacro:property name="wheel_mass" value="2" />
   <!-- end properties -->

Commit message: Fix model wheel size

File: src/rovr_description/urdf/rovr.urdf.xacro (robot description, xacro)
@@ -58,6 +58,6 @@
 	  <xacro:property name="base_mass" value="72.0" />
     <!--Part that extends from Body (Blue)-->
-    <xacro:property name="leg_height" value="0.0635"/>
-    <xacro:property name="leg_length" value="${base_length}"/>
+    <xacro:property name="leg_height" value=".1"/>
+    <xacro:property name="leg_length" value="0.5"/>
     <xacro:property name="leg_width" value="0.0508"/>
     <xacro:property name="leg_mass" value="4"/>
@@ -66,8 +66,8 @@
 	  <xacro:property name="leg_y_origin_to_axle" value="0.0254" />
 	  <xacro:property name="leg_axle_height" value="0.10535" />
-    <!--Rectangular representation of Drum (Purple)-->
-    <xacro:property name="drum_height" value="0.0635"/>
-    <xacro:property name="drum_length" value="0.110"/>
-    <xacro:property name="drum_width" value="${base_width-2*leg_width}"/>
+    <!-- Rectangular representation of Drum (Purple)-->
+    <xacro:property name="drum_height" value=".0300"/>
+    <xacro:property name="drum_length" value="${base_length+.01}"/>
+    <xacro:property name="drum_width" value=".110"/>
     <xacro:property name="drum_mass" value="2"/>
     <xacro:property name="drum_x_origin_to_base_origin" value=".195"/>

Commit message: remove drum from rovr model

File: src/rovr_description/urdf/rovr.urdf.xacro (robot description, xacro)
@@ -51,8 +51,8 @@
 <!-- Main dimensions: meters, kg, seconds, rads -->
 <!-- Rectangular Body Frame-->
-<xacro:property name="base_height" value=".500" /> <!--z-->
-<xacro:property name="base_length" value="0.500" /> <!--x-->
-<xacro:property name="base_width" value="0.7808" /> <!--y-->
-<xacro:property name="base_mass" value="72.0" />
+<xacro:property name="base_height" value=".500" />
+<xacro:property name="base_length" value="0.500" />
+<xacro:property name="base_width" value="0.7808" />
+<xacro:property name="base_mass" value="60.0" />
 <!--Part that extends from Body (Blue)-->
 <xacro:property name="leg_height" value=".1"/>
@@ -64,11 +64,4 @@
 <xacro:property name="leg_y_origin_to_axle" value="0.0254" />
 <xacro:property name="leg_axle_height" value="0.10535" />
-<!-- Rectangular representation of Drum (Purple)-->
-<xacro:property name="drum_height" value=".0300"/>
-<xacro:property name="drum_length" value="${base_length+.01}"/>
-<xacro:property name="drum_width" value=".110"/>
-<xacro:property name="drum_mass" value="2"/>
-<xacro:property name="drum_x_origin_to_base_origin" value=".195"/>
-<xacro:property name="drum_y_origin_to_base_origin" value="0"s/>
 <!-- End macros and properties -->
   <!-- End macros and properties -->
@@ -149,5 +142,5 @@
         <child link="right_leg" />
       </joint>
-      <!-- RIGHT_LEG represents the left of the drive train -->
+      <!-- RIGHT_LEG represents the right of the drive train -->
       <link name="right_leg">
         <!-- visual is the model shown in gazebo / rviz -->
@@ -179,41 +172,4 @@
       </gazebo>
     <!-- End right_leg_joint(right drive train) description -->
-    <!-- Attaching the drum to the robot frame -->
-    <!-- joint defines position relationship of the child to the parent-->
-    <joint name="drum_joint" type="fixed">
-		  <origin xyz="${drum_x_origin_to_base_origin} ${drum_y_origin_to_base_origin} ${-drum_height/2}" rpy="0 0 0" />
-		  <parent link="base_link" />
-		  <child link="drum" />
-	  </joint>
-    <!-- DRUM represents the digging wheel -->
-	  <link name="drum">
-      <!-- visual is the model shown in gazebo / rviz -->
-      <visual>
-        <origin xyz="0 0 0" rpy="0 0 0"/>
-        <geometry>
-          <box size=" ${drum_length} ${drum_width} ${drum_height}" />
-        </geometry>
-        <material name="purple"/>
-      </visual>
-      <!-- collision and inertial are used by the physics model used
-           in simulation -->
-      <collision>
-        <origin xyz="0 0 0" rpy="0 0 0"/>
-        <geometry>
-          <box size="${drum_length} ${drum_width} ${drum_width}"/>
-        </geometry>
-      </collision>
-      <inertial>
-        <origin xyz="0 0 0" rpy="0 0 0"/>
-        <mass value="${drum_mass}"/>
-        <box_inertial_matrix m="${drum_mass}" h="${drum_height}" l="${drum_length}" w="${drum_width}" />
-      </inertial>
-	  </link>
-    <!-- Gazebo element covers assigning values not handled by the URDF file format -->
-    <gazebo reference="drum">
-      <material>Gazebo/Purple</material>
-      <turnGravityOff>false</turnGravityOff>
-    </gazebo>
-    <!-- End drum description -->
   <!-- End links and joints -->
   <!-- The following represent extrusions from the frame and drivetrain
@@ -224,25 +180,5 @@
     <wheel prefix="back_left" leg="left_leg" x="-1" y="1"/>
     <wheel prefix="back_right" leg="right_leg" x="-1" y="-1"/>
-    <!-- extrusions for cameras / sensors -->
-    <extrusion prefix="front_left" x="1" y="1"/>
-    <extrusion prefix="front_right" x="1" y="-1"/>
-    <extrusion prefix="back_left" x="-1" y="1"/>
-    <extrusion prefix="back_right" x="-1" y="-1"/>
   <!-- End wheels and extrusions -->
-  <!-- The following represent the camera placementon the extrusions -->
-    <xacro:arg name="cameras" default="false"/>
-    <xacro:property name="useCams" value="$(arg cameras)"/>
-    <xacro:if value="${useCams == 'true'}">
-      <camera_macro number="1" y="1" extrusion="front_left_extrusion" spin="0"/>
-      <camera_macro number="2" y="-1" extrusion="front_right_extrusion" spin="0"/>
-      <camera_macro number="3" y="1" extrusion="back_left_extrusion" spin="${PI}"/>
-      <camera_macro number="4" y="-1" extrusion="back_right_extrusion" spin="${PI}"/>
-    </xacro:if>
-  <!-- End cameras -->
-  <!-- The following defines the positions of the IMU and Decawave sensors -->
-    <!-- imu and deca front left, back right. in front of extrusion -->
-    <imu number="1" x="1" y="1" extrusion="front_left_extrusion"/>
-    <imu number="2" x="1" y="-1" extrusion="back_right_extrusion"/>
-  <!-- End sensors -->
   <!-- skid steer plugin handles driving for us -->
 	<gazebo>
