Commit message: Update simulation to most recent master

File: src/rovr_description/urdf/rovr.urdf.xacro (robot description, xacro)
@@ -42,5 +42,5 @@
     <xacro:macro name="box_inertial_matrix" params="m l w h">
     	<inertia ixx="${(m*(w*w+h*h))/12.0}" ixy = "0.0" ixz = "0.0"
-       				 iyy="${(m*(l*l+h*h))/12.0}" iyz = "-1*base_width/20.0"
+       				 iyy="${(m*(l*l+h*h))/12.0}" iyz = "0.0"
        				 izz="${(m*(l*l+w*w))/12.0}" />
     </xacro:macro>
@@ -52,25 +52,22 @@
     </xacro:macro>
     <!-- Main dimensions: meters, kg, seconds, rads -->
-    <!-- Rectangular Body Frame (Gray)-->
-    <xacro:property name="base_height" value="0.500" /> <!--z-->
-	  <xacro:property name="base_length" value=".500" /> <!--x-->
-	  <xacro:property name="base_width" value="0.7808" /> <!--y-->
+    <xacro:property name="base_height" value="0.54" /> <!--z-->
+	  <xacro:property name="base_length" value="0.740" /> <!--x--> <!-- 0.864925 -->
+	  <xacro:property name="base_width" value="0.864925" /> <!--y--> <!-- 0.740 -->
 	  <xacro:property name="base_mass" value="72.0" />
-    <!--Part that extends from Body (Blue)-->
-    <xacro:property name="leg_height" value=".1"/>
-    <xacro:property name="leg_length" value="0.5"/>
+    <xacro:property name="leg_height" value="0.127"/>
+    <xacro:property name="leg_length" value="0.739775"/>
     <xacro:property name="leg_width" value="0.0508"/>
     <xacro:property name="leg_mass" value="4"/>
-    <!--Distance from Leg to Center-->
-    <xacro:property name="leg_x_origin_to_axle" value="${leg_length/2-.10835}" />
+    <xacro:property name="leg_x_origin_to_axle" value="${leg_length/2-.1778}" />
 	  <xacro:property name="leg_y_origin_to_axle" value="0.0254" />
 	  <xacro:property name="leg_axle_height" value="0.10535" />
-    <!-- Rectangular representation of Drum (Purple)-->
-    <xacro:property name="drum_height" value=".0300"/>
+    <xacro:property name="drum_height" value=".11809"/>
     <xacro:property name="drum_length" value="${base_length+.01}"/>
-    <xacro:property name="drum_width" value=".110"/>
+    <xacro:property name="drum_width" value=".34"/>
     <xacro:property name="drum_mass" value="2"/>
-    <xacro:property name="drum_x_origin_to_base_origin" value=".195"/>
-    <xacro:property name="drum_y_origin_to_base_origin" value="0"s/>
+    <xacro:property name="drum_y_origin_to_base_origin" value="${base_width/2-drum_width/2}"/>
+    <xacro:property name="realsense_front_offset" value="-0.0016"/>
+    <xacro:property name="realsense_back_offset" value="0.0429"/>
   <!-- End macros and properties -->
   <!-- The following links and joints define the robots components
@@ -183,5 +180,5 @@
     <!-- joint defines position relationship of the child to the parent-->
     <joint name="drum_joint" type="fixed">
-		  <origin xyz="${drum_x_origin_to_base_origin} ${drum_y_origin_to_base_origin} ${-drum_height/2}" rpy="0 0 0" />
+		  <origin xyz="0 ${drum_y_origin_to_base_origin} ${-drum_height/2}" rpy="0 0 0" />
 		  <parent link="base_link" />
 		  <child link="drum" />
@@ -232,5 +229,4 @@
   <!-- End wheels and extrusions -->
   <!-- The following represent the camera placement on the extrusions -->
-  <!--
     <xacro:arg name="cameras" default="false"/>
     <xacro:property name="useCams" value="$(arg cameras)"/>

File: src/rovr_description/urdf/wheel.urdf.xacro (robot description, xacro)
@@ -4,6 +4,6 @@
 	  <!-- Main dimensions: meters, kg, seconds, rads -->
 	  <xacro:property name="PI" value="3.141592653589793238462643383279502884197" />
-	  <xacro:property name="wheel_width" value=".1" />
-	  <xacro:property name="wheel_radius" value="0.1225" />
+	  <xacro:property name="wheel_width" value=".15" />
+	  <xacro:property name="wheel_radius" value=".18035" />
 	  <xacro:property name="wheel_mass" value="2" />
   <!-- end properties -->

Commit message: Update robot model to new dimensions

File: src/rovr_description/urdf/rovr.urdf.xacro (robot description, xacro)
@@ -52,14 +52,14 @@
     </xacro:macro>
     <!-- Main dimensions: meters, kg, seconds, rads -->
-    <xacro:property name="base_height" value="0.54" /> <!--z-->
-	  <xacro:property name="base_length" value="0.740" /> <!--x--> <!-- 0.864925 -->
-	  <xacro:property name="base_width" value="0.864925" /> <!--y--> <!-- 0.740 -->
-	  <xacro:property name="base_mass" value="72.0" />
-    <xacro:property name="leg_height" value="0.127"/>
-    <xacro:property name="leg_length" value="0.739775"/>
-    <xacro:property name="leg_width" value="0.0508"/>
-    <xacro:property name="leg_mass" value="4"/>
-    <xacro:property name="leg_x_origin_to_axle" value="${leg_length/2-.1778}" />
-	  <xacro:property name="leg_y_origin_to_axle" value="0.0254" />
+    <xacro:property name="base_height" value="0.495" /> <!--z-->
+	  <xacro:property name="base_length" value="0.495" /> <!--x--> <!-- 0.864925 -->
+	  <xacro:property name="base_width" value="0.8316" /> <!--y--> <!-- 0.740 -->
+	  <xacro:property name="base_mass" value="36.0" />
+    <xacro:property name="leg_height" value="0.140"/>
+    <xacro:property name="leg_length" value="0.3934"/>
+    <xacro:property name="leg_width" value="0.037"/>
+    <xacro:property name="leg_mass" value="0.01"/>
+    <xacro:property name="leg_x_origin_to_axle" value="0.1275" />
+	  <xacro:property name="leg_y_origin_to_axle" value="0" />
 	  <xacro:property name="leg_axle_height" value="0.10535" />
     <xacro:property name="drum_height" value=".11809"/>
@@ -68,4 +68,5 @@
     <xacro:property name="drum_mass" value="2"/>
     <xacro:property name="drum_y_origin_to_base_origin" value="${base_width/2-drum_width/2}"/>
+    <xacro:property name="leg_y" value="-0.075" />
     <xacro:property name="realsense_front_offset" value="-0.0016"/>
     <xacro:property name="realsense_back_offset" value="0.0429"/>
@@ -75,5 +76,15 @@
     <!-- BASE_LINK represent the frame of the robot -->
 	    <link name="base_link">
-		    <!-- visual is the model shown in gazebo / rviz -->
+		    <visual>
+			    <origin xyz="0 0 ${base_height/2.0}" rpy="0 0 0"/>
+			    <geometry>
+				    <box size=" ${base_length} ${base_width} ${base_height}" />
+			    </geometry>
+			    <material name="grey"/>
+		    </visual>
+	    </link>
+      <!-- Gazebo doesn't support base_link with inertia-->
+      <link name="dummy_mass">
+        <!-- visual is the model shown in gazebo / rviz -->
 		    <visual>
 			    <origin xyz="0 0 ${base_height/2.0}" rpy="0 0 0"/>
@@ -91,10 +102,15 @@
 			    </geometry>
 		    </collision>
-		    <inertial>
+        <inertial>
 			    <origin xyz="0 0 ${base_height/2.0}" rpy="0 0 0"/>
 			    <mass value="${base_mass}"/>
 			    <box_inertial_matrix m="${base_mass}" h="${base_height}" l="${base_length}" w="${base_width}" />
 		    </inertial>
-	    </link>
+      </link>
+      <joint name="base_dummy_joint" type="fixed">
+		    <origin xyz="0 0 0" rpy="0 0 0" />
+		    <parent link="base_link" />
+		    <child link="dummy_mass" />
+	    </joint>
       <!-- Gazebo element covers assigning values not handled by the URDF file format -->
       <gazebo reference="base_link">
@@ -106,5 +122,5 @@
       <!-- joint defines position relationship of the child to the parent-->
       <joint name="left_leg_joint" type="fixed">
-		    <origin xyz="0 ${base_width/2-leg_width/2} ${-leg_height}" rpy="0 0 0" />
+		    <origin xyz="0 ${base_width/2-leg_width/2} ${leg_y}" rpy="0 0 0" />
 		    <parent link="base_link" />
 		    <child link="left_leg" />
@@ -143,5 +159,5 @@
       <!-- joint defines position relationship of the child to the parent-->
       <joint name="right_leg_joint" type="fixed">
-        <origin xyz="0 ${-base_width/2+leg_width/2} ${-leg_height}" rpy="0 0 0" />
+        <origin xyz="0 ${-base_width/2+leg_width/2} ${leg_y}" rpy="0 0 0" />
         <parent link="base_link" />
         <child link="right_leg" />
@@ -177,41 +193,4 @@
       </gazebo>
     <!-- End right_leg_joint(right drive train) description -->
-    <!-- Attaching the drum to the robot frame -->
-    <!-- joint defines position relationship of the child to the parent-->
-    <joint name="drum_joint" type="fixed">
-		  <origin xyz="0 ${drum_y_origin_to_base_origin} ${-drum_height/2}" rpy="0 0 0" />
-		  <parent link="base_link" />
-		  <child link="drum" />
-	  </joint>
-    <!-- DRUM represents the digging wheel -->
-	  <link name="drum">
-      <!-- visual is the model shown in gazebo / rviz -->
-      <visual>
-        <origin xyz="0 0 0" rpy="0 0 0"/>
-        <geometry>
-          <box size=" ${drum_length} ${drum_width} ${drum_height}" />
-        </geometry>
-        <material name="purple"/>
-      </visual>
-      <!-- collision and inertial are used by the physics model used
-           in simulation -->
-      <collision>
-        <origin xyz="0 0 0" rpy="0 0 0"/>
-        <geometry>
-          <box size="${drum_length} ${drum_width} ${drum_width}"/>
-        </geometry>
-      </collision>
-      <inertial>
-        <origin xyz="0 0 0" rpy="0 0 0"/>
-        <mass value="${drum_mass}"/>
-        <box_inertial_matrix m="${drum_mass}" h="${drum_height}" l="${drum_length}" w="${drum_width}" />
-      </inertial>
-	  </link>
-    <!-- Gazebo element covers assigning values not handled by the URDF file format -->
-    <gazebo reference="drum">
-      <material>Gazebo/Purple</material>
-      <turnGravityOff>false</turnGravityOff>
-    </gazebo>
-    <!-- End drum description -->
   <!-- End links and joints -->
   <!-- The following represent extrusions from the frame and drivetrain

File: src/rovr_description/urdf/sensors/realsense.urdf.xacro (robot description, xacro)
@@ -4,6 +4,6 @@
   <xacro:include filename="$(find rovr_description)/urdf/_d435.urdf.xacro"/>
   <!-- Main dimensions: meters, kg, seconds, rads -->
-  <xacro:property name="realsense_vertical_from_base" value = "0.4763" />
-  <xacro:property name="realsense_horizontal_from_base" value = "0.3493" />
+  <xacro:property name="realsense_vertical_from_base" value = "0.371" />
+  <xacro:property name="realsense_horizontal_from_base" value = "0.248" />
   <xacro:property name="realsense_angle" value="0.55" /> <!--rad from horizontal, + = downward-->
   <xacro:property name="PI" value="3.1415926535897931" />

File: src/rovr_description/urdf/wheel.urdf.xacro (robot description, xacro)
@@ -4,6 +4,6 @@
 	  <!-- Main dimensions: meters, kg, seconds, rads -->
 	  <xacro:property name="PI" value="3.141592653589793238462643383279502884197" />
-	  <xacro:property name="wheel_width" value=".15" />
-	  <xacro:property name="wheel_radius" value=".18035" />
+	  <xacro:property name="wheel_width" value=".10" />
+	  <xacro:property name="wheel_radius" value=".120" />
 	  <xacro:property name="wheel_mass" value="2" />
   <!-- end properties -->
@@ -35,5 +35,5 @@
 			<parent link="${leg}" />
 			<child 	link="${prefix}_wheel" />
-      <origin xyz="${x*leg_x_origin_to_axle} ${y*(wheel_radius/2+leg_width/4)} ${leg_axle_height-leg_height/2}" rpy="0 0 0"/>
+      <origin xyz="${x*leg_x_origin_to_axle} ${y*(wheel_radius/2+leg_width/4)} ${leg_axle_height-leg_height/2-0.01}" rpy="0 0 0"/>
       <dynamics damping="0.5" friction="0.1"/> <!-- get real later N*m*s/rad damp N*m friction-->
       <limit effort="1000" velocity="10"/> <!-- simmulate motors, max velocity and max joint effort -->
